Commit message: Mostly working

File: model/parameters.urdf.xacro (robot description, xacro)
@@ -10,5 +10,5 @@
 <xacro:property name="joint_lower_limit" value="${-pi/2}"/>
 <xacro:property name="joint_upper_limit" value="${pi/2}"/>
-<xacro:property name="end_effector_radius" value="0.3"/>
+<xacro:property name="end_effector_radius" value="0.2"/>
 <xacro:property name="end_effector_depth" value="0.03"/>
 <xacro:property name="base_mass" value="0.1"/>
