Commit message: Fixed angle origins

File: model/delta_end_effector.urdf.xacro (robot description, xacro)
@@ -19,5 +19,5 @@
 <!-- ===== ACTUAL END EFFECTOR ===== -->
 <joint name="lower_bot_1_to_virtual_end_effector_offset" type="revolute">
-    <axis xyz="0 1 0"/>
+    <axis xyz="0 -1 0"/>
     <limit
         effort="1000.0"
@@ -27,6 +27,6 @@
     />
     <origin
-        rpy="${pi} 0 0"
-        xyz="${end_effector_radius} ${-lower_horizontal_length/2} 0"
+        rpy="0 0 0"
+        xyz="0 ${-lower_horizontal_length/2} 0"
     />
     <parent link="lower_bot_1"/>
@@ -46,5 +46,5 @@
 </link>
 <joint name="virtual_end_effector_offset_to_end_effector" type="fixed">
-    <origin rpy="0 0 0" xyz="0 0 0"/>
+    <origin rpy="0 0 0" xyz="${end_effector_radius} 0 0"/>
     <parent link="virtual_end_effector_offset"/>
     <child link="end_effector"/>

File: model/delta_lower.urdf.xacro (robot description, xacro)
@@ -12,5 +12,5 @@
     />
     <origin
-        rpy="0 0 0"
+        rpy="0 0 ${pi}"
         xyz="${upper_length} 0 0"
     />
@@ -65,5 +65,5 @@
     />
     <origin
-        rpy="0 ${pi/2} 0"
+        rpy="0 0 0"
         xyz="0 ${lower_horizontal_length/2} 0"
     />
@@ -124,5 +124,5 @@
     />
     <origin
-        rpy="0 ${pi/2} 0"
+        rpy="0 0 0"
         xyz="0 ${-lower_horizontal_length/2} 0"
     />

Commit message: Finished urdf model

File: model/delta_end_effector.urdf.xacro (robot description, xacro)
@@ -1,21 +1,5 @@
 <?xml version="1.0"?>
 <robot xmlns:xacro="http://www.ros.org/wiki/xacro" name="delta">
-<!-- ===== VIRTUAL END EFFECTORS ===== -->
-<!--
-<xacro:macro name="link_virtual_end_effector" params="number">
-<link name="virtual_end_effector_${number}">
-    <visual>
-        <geometry>
-            <sphere radius="break_indicator_radius"/>
-        </geometry>
-        <material name="break_indicator"/>
-    </visual>
-</link>
-</xacro:macro>
-<xacro:link_virtual_end_effector number="1"/>
-<xacro:link_virtual_end_effector number="2"/>
-<xacro:link_virtual_end_effector number="3"/>
--->
-<!-- ===== ACTUAL END EFFECTOR ===== -->
+<!-- ===== END EFFECTOR ===== -->
 <joint name="lower_bot_1_to_virtual_end_effector_offset" type="revolute">
     <axis xyz="0 -1 0"/>

File: model/delta_lower_virtual.urdf.xacro (robot description, xacro)
@@ -1,3 +1,106 @@
 <?xml version="1.0"?>
 <robot xmlns:xacro="http://www.ros.org/wiki/xacro" name="delta">
+<!-- ===== VIRTUAL_LOWER_OFFSET ===== -->
+<xacro:macro name="joint_upper_to_virtual_lower_offset" params="number">
+<joint name="upper_to_virtual_lower_offset_${number}" type="revolute">
+    <axis xyz="0 1 0"/>
+    <limit
+        effort="1000.0"
+        lower="${-pi/2}"
+        upper="${pi/2}"
+        velocity="0.5"
+    />
+    <origin
+        rpy="0 0 ${pi}"
+        xyz="${upper_length} 0 0"
+    />
+    <parent link="upper_${number}"/>
+    <child link="virtual_lower_offset_${number}"/>
+</joint>
+</xacro:macro>
+<xacro:joint_upper_to_virtual_lower_offset number="1"/>
+<xacro:joint_upper_to_virtual_lower_offset number="2"/>
+<xacro:joint_upper_to_virtual_lower_offset number="3"/>
+<xacro:macro name="link_virtual_lower_offset" params="number">
+<link name="virtual_lower_offset_${number}">
+<visual>
+    <geometry>
+        <cylinder length="${end_effector_radius}" radius="${lower_radius}"/>
+    </geometry>
+    <origin
+        rpy="0 ${pi/2} 0"
+        xyz="${end_effector_radius/2} 0 0"
+    />
+    <material name="virtual_link"/>
+</visual>
+</link>
+</xacro:macro>
+<xacro:link_virtual_lower_offset number="1"/>
+<xacro:link_virtual_lower_offset number="2"/>
+<xacro:link_virtual_lower_offset number="3"/>
+<!-- ===== VIRTUAL_LOWER ===== -->
+<xacro:macro name="joint_virtual_lower_offset_to_virtual_lower" params="number">
+<joint name="virtual_lower_offset_to_virtual_lower_${number}" type="revolute">
+    <axis xyz="0 1 0"/>
+    <limit
+        effort="1000.0"
+        lower="${-pi/2}"
+        upper="${pi/2}"
+        velocity="0.5"
+    />
+    <origin
+        rpy="0 0 0"
+        xyz="${end_effector_radius} 0 0"
+    />
+    <parent link="virtual_lower_offset_${number}"/>
+    <child link="virtual_lower_${number}"/>
+</joint>
+</xacro:macro>
+<xacro:joint_virtual_lower_offset_to_virtual_lower number="1"/>
+<xacro:joint_virtual_lower_offset_to_virtual_lower number="2"/>
+<xacro:joint_virtual_lower_offset_to_virtual_lower number="3"/>
+<xacro:macro name="link_virtual_lower" params="number">
+<link name="virtual_lower_${number}">
+<visual>
+    <geometry>
+        <cylinder length="${lower_vertical_length}" radius="${lower_radius}"/>
+    </geometry>
+    <origin
+        rpy="0 ${pi/2} 0"
+        xyz="${lower_vertical_length/2} 0 0"
+    />
+    <material name="virtual_link"/>
+</visual>
+</link>
+</xacro:macro>
+<xacro:link_virtual_lower number="1"/>
+<xacro:link_virtual_lower number="2"/>
+<xacro:link_virtual_lower number="3"/>
+<!-- ===== VIRTUAL END EFFECTORS ===== -->
+<xacro:macro name="joint_virtual_lower_to_virtual_end_effector" params="number">
+<joint name="virtual_lower_to_virtual_end_effector_${number}" type="fixed">
+    <origin
+        rpy="0 0 0"
+        xyz="${lower_vertical_length} 0 0"
+    />
+    <parent link="virtual_lower_${number}"/>
+    <child link="virtual_end_effector_${number}"/>
+</joint>
+</xacro:macro>
+<xacro:joint_virtual_lower_to_virtual_end_effector number="1"/>
+<xacro:joint_virtual_lower_to_virtual_end_effector number="2"/>
+<xacro:joint_virtual_lower_to_virtual_end_effector number="3"/>
+<xacro:macro name="link_virtual_end_effector" params="number">
+<link name="virtual_end_effector_${number}">
+    <visual>
+        <geometry>
+            <sphere radius="${break_indicator_radius}"/>
+        </geometry>
+        <material name="break_indicator"/>
+    </visual>
+</link>
+</xacro:macro>
+<xacro:link_virtual_end_effector number="1"/>
+<xacro:link_virtual_end_effector number="2"/>
+<xacro:link_virtual_end_effector number="3"/>
 </robot>

File: model/parameters.urdf.xacro (robot description, xacro)
@@ -2,8 +2,8 @@
 <robot xmlns:xacro="http://www.ros.org/wiki/xacro" name="delta_parameters">
 <xacro:property name="base_radius" value="0.3"/>
-<xacro:property name="base_depth" value="0.1"/>
+<xacro:property name="base_depth" value="0.02"/>
 <xacro:property name="upper_length" value="0.3"/>
-<xacro:property name="upper_radius" value="0.03"/>
-<xacro:property name="lower_radius" value="0.03"/>
+<xacro:property name="upper_radius" value="0.01"/>
+<xacro:property name="lower_radius" value="0.01"/>
 <xacro:property name="lower_horizontal_length" value="0.4"/>
 <xacro:property name="lower_vertical_length" value="0.6"/>
@@ -17,4 +17,4 @@
 <xacro:property name="lower_vertical_mass" value="0.04"/>
 <xacro:property name="end_effector_mass" value="0.05"/>
-<xacro:property name="break_indicator_radius" value="0.05"/>
+<xacro:property name="break_indicator_radius" value="0.04"/>
 </robot>

Commit message: Fixed urdf, added simple constraints

File: model/delta_end_effector.urdf.xacro (robot description, xacro)
@@ -18,14 +18,4 @@
 </joint>
 <link name="virtual_end_effector_offset">
-    <visual>
-        <geometry>
-            <cylinder
-                length="${end_effector_radius}"
-                radius="${end_effector_depth}"
-            />
-        </geometry>
-        <origin rpy="0 ${pi/2} 0" xyz="${end_effector_radius/2} 0 0"/>
-        <material name="virtual_link"/>
-    </visual>
 </link>
 <joint name="virtual_end_effector_offset_to_end_effector" type="fixed">

File: model/delta_lower.urdf.xacro (robot description, xacro)
@@ -175,5 +175,5 @@
 <xacro:macro name="joint_lower_left_to_lower_bot" params="number">
 <joint name="lower_left_to_lower_bot_${number}" type="revolute">
-    <axis xyz="0 0 1"/>
+    <axis xyz="0 0 -1"/>
     <limit
         effort="1000.0"

File: model/delta_lower_virtual.urdf.xacro (robot description, xacro)
@@ -1,7 +1,7 @@
 <?xml version="1.0"?>
 <robot xmlns:xacro="http://www.ros.org/wiki/xacro" name="delta">
-<!-- ===== VIRTUAL_LOWER_OFFSET ===== -->
-<xacro:macro name="joint_upper_to_virtual_lower_offset" params="number">
-<joint name="upper_to_virtual_lower_offset_${number}" type="revolute">
+<!-- ===== PSEUDO_ELBOW_OFFSET ===== -->
+<xacro:macro name="joint_upper_to_pseudo_elbow_offset" params="number">
+<joint name="upper_to_pseudo_elbow_offset_${number}" type="revolute">
     <axis xyz="0 1 0"/>
     <limit
@@ -16,12 +16,12 @@
     />
     <parent link="upper_${number}"/>
-    <child link="virtual_lower_offset_${number}"/>
+    <child link="pseudo_elbow_offset_${number}"/>
 </joint>
 </xacro:macro>
-<xacro:joint_upper_to_virtual_lower_offset number="1"/>
-<xacro:joint_upper_to_virtual_lower_offset number="2"/>
-<xacro:joint_upper_to_virtual_lower_offset number="3"/>
-<xacro:macro name="link_virtual_lower_offset" params="number">
-<link name="virtual_lower_offset_${number}">
+<xacro:joint_upper_to_pseudo_elbow_offset number="1"/>
+<xacro:joint_upper_to_pseudo_elbow_offset number="2"/>
+<xacro:joint_upper_to_pseudo_elbow_offset number="3"/>
+<xacro:macro name="link_pseudo_elbow_offset" params="number">
+<link name="pseudo_elbow_offset_${number}">
 <visual>
     <geometry>
@@ -36,10 +36,10 @@
 </link>
 </xacro:macro>
-<xacro:link_virtual_lower_offset number="1"/>
-<xacro:link_virtual_lower_offset number="2"/>
-<xacro:link_virtual_lower_offset number="3"/>
-<!-- ===== VIRTUAL_LOWER ===== -->
-<xacro:macro name="joint_virtual_lower_offset_to_virtual_lower" params="number">
-<joint name="virtual_lower_offset_to_virtual_lower_${number}" type="revolute">
+<xacro:link_pseudo_elbow_offset number="1"/>
+<xacro:link_pseudo_elbow_offset number="2"/>
+<xacro:link_pseudo_elbow_offset number="3"/>
+<!-- ===== PSEUDO_ELBOW ===== -->
+<xacro:macro name="joint_pseudo_elbow_offset_to_pseudo_elbow" params="number">
+<joint name="pseudo_elbow_offset_to_pseudo_elbow_${number}" type="revolute">
     <axis xyz="0 1 0"/>
     <limit
@@ -53,11 +53,39 @@
         xyz="${end_effector_radius} 0 0"
     />
-    <parent link="virtual_lower_offset_${number}"/>
+    <parent link="pseudo_elbow_offset_${number}"/>
+    <child link="pseudo_elbow_${number}"/>
+</joint>
+</xacro:macro>
+<xacro:joint_pseudo_elbow_offset_to_pseudo_elbow number="1"/>
+<xacro:joint_pseudo_elbow_offset_to_pseudo_elbow number="2"/>
+<xacro:joint_pseudo_elbow_offset_to_pseudo_elbow number="3"/>
+<xacro:macro name="link_pseudo_elbow" params="number">
+<link name="pseudo_elbow_${number}">
+</link>
+</xacro:macro>
+<xacro:link_pseudo_elbow number="1"/>
+<xacro:link_pseudo_elbow number="2"/>
+<xacro:link_pseudo_elbow number="3"/>
+<!-- ===== VIRTUAL_LOWER ===== -->
+<xacro:macro name="joint_pseudo_elbow_to_virtual_lower" params="number">
+<joint name="pseudo_elbow_to_virtual_lower_${number}" type="revolute">
+    <axis xyz="0 0 1"/>
+    <limit
+        effort="1000.0"
+        lower="${-pi/2}"
+        upper="${pi/2}"
+        velocity="0.5"
+    />
+    <origin
+        rpy="0 0 0"
+        xyz="0 0 0"
+    />
+    <parent link="pseudo_elbow_${number}"/>
     <child link="virtual_lower_${number}"/>
 </joint>
 </xacro:macro>
-<xacro:joint_virtual_lower_offset_to_virtual_lower number="1"/>
-<xacro:joint_virtual_lower_offset_to_virtual_lower number="2"/>
-<xacro:joint_virtual_lower_offset_to_virtual_lower number="3"/>
+<xacro:joint_pseudo_elbow_to_virtual_lower number="1"/>
+<xacro:joint_pseudo_elbow_to_virtual_lower number="2"/>
+<xacro:joint_pseudo_elbow_to_virtual_lower number="3"/>
 <xacro:macro name="link_virtual_lower" params="number">
 <link name="virtual_lower_${number}">

File: model/materials.urdf.xacro (robot description, xacro)
@@ -2,5 +2,5 @@
 <robot xmlns:xacro="http://www.ros.org/wiki/xacro" name="delta_materials">
 <material name="break_indicator">
-    <color rgba="0 0 0 1"/>
+    <color rgba="1 0 0 1"/>
 </material>
 <material name="physical_link">

File: model/parameters.urdf.xacro (robot description, xacro)
@@ -17,4 +17,4 @@
 <xacro:property name="lower_vertical_mass" value="0.04"/>
 <xacro:property name="end_effector_mass" value="0.05"/>
-<xacro:property name="break_indicator_radius" value="0.04"/>
+<xacro:property name="break_indicator_radius" value="0.03"/>
 </robot>

Commit message: Improvements to urdf

File: model/delta_end_effector.urdf.xacro (robot description, xacro)
@@ -4,5 +4,4 @@
 <xacro:macro name="joint_end_effector" params="number yaw">
 <joint name="lower_${number}_end_to_end_effector" type="fixed">
-    <origin rpy="0 0 0" xyz="${end_effector_radius} 0 0"/>
     <origin
         rpy="0 ${pi} ${yaw}"
@@ -19,23 +18,62 @@
 </gazebo>
 <link name="end_effector">
-    <visual>
-        <geometry>
-            <cylinder
-                length="${end_effector_depth}"
-                radius="${end_effector_radius}"
-            />
-        </geometry>
-        <origin rpy="0 0 0" xyz="0 0 0"/>
-        <material name="end_effector"/>
-    </visual>
-    <collision>
-        <geometry>
-            <cylinder
-                length="${end_effector_depth}"
-                radius="${end_effector_radius}"
-            />
-        </geometry>
-        <origin rpy="0 0 0" xyz="0 0 0"/>
-    </collision>
+<visual>
+    <geometry>
+        <cylinder
+            length="${end_effector_depth}"
+            radius="${end_effector_radius}"
+        />
+    </geometry>
+    <origin rpy="0 0 0" xyz="0 0 0"/>
+    <material name="end_effector"/>
+</visual>
+<collision>
+    <geometry>
+        <cylinder
+            length="${end_effector_depth}"
+            radius="${end_effector_radius}"
+        />
+    </geometry>
+    <origin rpy="0 0 0" xyz="0 0 0"/>
+</collision>
+<visual>
+    <geometry>
+        <cylinder length="${lower_width}" radius="${end_effector_depth/2}" />
+    </geometry>
+    <origin xyz="${end_effector_radius} 0 0" rpy="0 ${pi/2} ${pi/2}" />
+    <material name="end_effector"/>
+</visual>
+<collision>
+    <geometry>
+        <cylinder length="${lower_width}" radius="${end_effector_depth/2}" />
+    </geometry>
+    <origin xyz="${end_effector_radius} 0 0" rpy="0 ${pi/2} ${pi/2}" />
+</collision>
+<visual>
+    <geometry>
+        <cylinder length="${lower_width}" radius="${end_effector_depth/2}" />
+    </geometry>
+    <origin xyz="${cos(pi*2/3)*end_effector_radius} ${sin(pi*2/3)*end_effector_radius} 0" rpy="0 ${pi/2} ${pi*7/6}" />
+    <material name="end_effector"/>
+</visual>
+<collision>
+    <geometry>
+        <cylinder length="${lower_width}" radius="${end_effector_depth/2}" />
+    </geometry>
+    <origin xyz="${cos(pi*2/3)*end_effector_radius} ${sin(pi*2/3)*end_effector_radius} 0" rpy="0 ${pi/2} ${pi*7/6}" />
+</collision>
+<visual>
+    <geometry>
+        <cylinder length="${lower_width}" radius="${end_effector_depth/2}" />
+    </geometry>
+    <origin xyz="${cos(pi*4/3)*end_effector_radius} ${sin(pi*4/3)*end_effector_radius} 0" rpy="0 ${pi/2} ${pi*11/6}" />
+    <material name="end_effector"/>
+</visual>
+<collision>
+    <geometry>
+        <cylinder length="${lower_width}" radius="${end_effector_depth/2}" />
+    </geometry>
+    <origin xyz="${cos(pi*4/3)*end_effector_radius} ${sin(pi*4/3)*end_effector_radius} 0" rpy="0 ${pi/2} ${pi*11/6}" />
+</collision>
 </link>
 </robot>

File: model/delta_upper.urdf.xacro (robot description, xacro)
@@ -56,4 +56,29 @@
     />
 </collision>
+<visual>
+    <geometry>
+        <cylinder
+            length="${lower_width}"
+            radius="${upper_radius}"
+        />
+    </geometry>
+    <origin
+        xyz="${upper_length} 0 0"
+        rpy="${pi/2} 0 0"
+    />
+    <material name="upper"/>
+</visual>
+<collision>
+    <geometry>
+        <cylinder
+            length="${lower_width}"
+            radius="${upper_radius}"
+        />
+    </geometry>
+    <origin
+        xyz="${upper_length} 0 0"
+        rpy="${pi/2} 0 0"
+    />
+</collision>
 </link>
 </xacro:macro>

Commit message: FK works

File: model/delta_end_effector.urdf.xacro (robot description, xacro)
@@ -2,6 +2,6 @@
 <robot xmlns:xacro="http://www.ros.org/wiki/xacro" name="delta">
 <!-- ===== END EFFECTOR ===== -->
-<xacro:macro name="joint_end_effector" params="number yaw">
-<joint name="lower_${number}_end_to_end_effector" type="fixed">
+<xacro:macro name="chain_end" params="number yaw">
+<joint name="lower_end_to_chain_end_${number}" type="fixed">
     <origin
         rpy="0 ${pi} ${yaw}"
@@ -9,11 +9,23 @@
     />
     <parent link="lower_${number}_end"/>
+    <child link="chain_${number}_end"/>
+</joint>
+<link name="chain_${number}_end">
+</link>
+</xacro:macro>
+<xacro:chain_end number="1" yaw="0"/>
+<xacro:chain_end number="2" yaw="${pi*2/3}"/>
+<xacro:chain_end number="3" yaw="${pi*4/3}"/>
+<xacro:macro name="joint_chain_end_to_end_effector" params="number">
+<joint name="chain_${number}_end_to_end_effector" type="fixed">
+    <origin xyz="0 0 0" rpy="0 0 0"/>
+    <parent link="chain_${number}_end"/>
     <child link="end_effector"/>
 </joint>
 </xacro:macro>
-<xacro:joint_end_effector number="1" yaw="0"/>
+<xacro:joint_chain_end_to_end_effector number="1"/>
 <gazebo>
-<xacro:joint_end_effector number="2" yaw="${pi*2/3}"/>
-<xacro:joint_end_effector number="3" yaw="${pi*4/3}"/>
+<xacro:joint_chain_end_to_end_effector number="2"/>
+<xacro:joint_chain_end_to_end_effector number="3"/>
 </gazebo>
 <link name="end_effector">
