Commit message: Publishes relative TFs correctly, now need to set the dependent joint values

File: model/delta.urdf.xacro (robot description, xacro)
@@ -407,7 +407,7 @@
     </visual>
 </link>
-<joint name="end_effector_virtual_joint" type="floating">
-    <origin rpy="0 0 0" xyz="0 0 0"/>
-    <parent link="base"/>
+<joint name="end_effector_1_to_end_effector" type="fixed">
+    <origin rpy="0 0 0" xyz="${end_effector_radius} 0 0"/>
+    <parent link="end_effector_1"/>
     <child link="end_effector"/>
 </joint>

Commit message: Restructed urdf

File: model/delta.urdf.xacro (robot description, xacro)
@@ -2,415 +2,10 @@
 <robot xmlns:xacro="http://www.ros.org/wiki/xacro" name="delta">
 <xacro:include filename="parameters.urdf.xacro"/>
-<!-- gives inertia of AAC cylinder. Provide rpy to rotate the inertial frame
-such that Z is aligned with the axis of the cylinder-->
-<xacro:macro name="cylinder_inertial" params="mass radius length rpy">
-<inertial>
-    <origin rpy="${rpy}" xyz="0 0 0"/>
-    <mass value="${mass}"/>
-    <inertia
-        ixx="${mass*(radius**2/4 + length**2/12)}"
-        iyy="${mass*(radius**2/4 + length**2/12)}"
-        izz="${mass*(radius**2/2)}"
-        ixy="0" ixz="0" iyz="0"
-    />
-</inertial>
-</xacro:macro>
-<xacro:macro name="link_base">
-<link name="base">
-<!-- root link doesn't need inertia -->
-<visual>
-    <geometry>
-        <cylinder
-            length="${base_depth}"
-            radius="${base_radius}"
-        />
-    </geometry>
-</visual>
-<collision>
-    <geometry>
-        <cylinder
-            length="${base_depth}"
-            radius="${base_radius}"
-        />
-    </geometry>
-</collision>
-</link>
-</xacro:macro>
-<xacro:link_base/>
-<xacro:macro name="joint_base_to_upper" params="number yaw">
-<joint name="base_to_upper_${number}" type="revolute">
-    <axis xyz="0 1 0"/>
-    <limit
-        effort="1000.0"
-        lower="${joint_lower_limit}"
-        upper="${joint_upper_limit}"
-        velocity="0.5"
-    />
-    <origin
-        rpy="0 0 ${yaw}"
-        xyz="${cos(yaw)*base_radius} ${sin(yaw)*base_radius} 0"
-    />
-    <parent link="base"/>
-    <child link="upper_${number}"/>
-</joint>
-</xacro:macro>
-<xacro:joint_base_to_upper number="1" yaw="0"/>
-<xacro:joint_base_to_upper number="2" yaw="${pi*2/3}"/>
-<xacro:joint_base_to_upper number="3" yaw="${-pi*2/3}"/>
-<xacro:macro name="link_upper" params="number">
-<link name="upper_${number}">
-<xacro:cylinder_inertial
-    mass="${upper_mass}"
-    radius="${upper_radius}"
-    length="${upper_length}"
-    rpy="0 ${pi/2} 0"
-/>
-<visual>
-    <geometry>
-        <cylinder
-            length="${upper_length}"
-            radius="${upper_radius}"
-        />
-    </geometry>
-    <origin
-        xyz="${upper_length/2} 0 0"
-        rpy="0 ${pi/2} 0"
-    />
-</visual>
-<collision>
-    <geometry>
-        <cylinder
-            length="${upper_length}"
-            radius="${upper_radius}"
-        />
-    </geometry>
-    <origin
-        xyz="${upper_length/2} 0 0"
-        rpy="0 ${pi/2} 0"
-    />
-</collision>
-</link>
-</xacro:macro>
-<xacro:link_upper number="1"/>
-<xacro:link_upper number="2"/>
-<xacro:link_upper number="3"/>
-<xacro:macro name="joint_upper_to_elbow" params="number">
-<joint name="upper_to_elbow_${number}" type="revolute">
-    <axis xyz="0 1 0"/>
-    <limit
-        effort="1000.0"
-        lower="${-pi/2}"
-        upper="${pi/2}"
-        velocity="0.5"
-    />
-    <origin
-        rpy="0 0 0"
-        xyz="${upper_length} 0 0"
-    />
-    <parent link="upper_${number}"/>
-    <child link="elbow_${number}"/>
-</joint>
-</xacro:macro>
-<xacro:joint_upper_to_elbow number="1"/>
-<xacro:joint_upper_to_elbow number="2"/>
-<xacro:joint_upper_to_elbow number="3"/>
-<xacro:macro name="link_elbow" params="number">
-<link name="elbow_${number}">
-<xacro:cylinder_inertial
-    mass="${elbow_mass}"
-    radius="${elbow_radius}"
-    length="${upper_length}"
-    rpy="0 ${pi/2} ${pi/2}"
-/>
-<visual>
-    <geometry>
-        <cylinder length="${elbow_length}" radius="${elbow_radius}"/>
-    </geometry>
-    <origin
-        rpy="0 ${pi/2} ${pi/2}"
-        xyz="0 0 0"
-    />
-</visual>
-<collision>
-    <geometry>
-        <cylinder length="${elbow_length}" radius="${elbow_radius}"/>
-    </geometry>
-    <origin
-        rpy="0 ${pi/2} ${pi/2}"
-        xyz="0 0 0"
-    />
-</collision>
-</link>
-</xacro:macro>
-<xacro:link_elbow number="1"/>
-<xacro:link_elbow number="2"/>
-<xacro:link_elbow number="3"/>
-<xacro:macro name="joint_elbow_to_lower_left" params="number">
-<joint name="elbow_to_lower_left_${number}" type="revolute">
-    <axis xyz="0 0 1"/>
-    <limit
-        effort="1000.0"
-        lower="${-pi/2}"
-        upper="${pi/2}"
-        velocity="0.5"
-    />
-    <origin
-        rpy="0 ${pi/2} 0"
-        xyz="0 ${elbow_length/2} 0"
-    />
-    <parent link="elbow_${number}"/>
-    <child link="lower_left_${number}"/>
-</joint>
-</xacro:macro>
-<xacro:joint_elbow_to_lower_left number="1"/>
-<xacro:joint_elbow_to_lower_left number="2"/>
-<xacro:joint_elbow_to_lower_left number="3"/>
-<xacro:macro name="link_lower_left" params="number">
-<link name="lower_left_${number}">
-<xacro:cylinder_inertial
-    mass="${lower_mass}"
-    radius="${lower_radius}"
-    length="${lower_length}"
-    rpy="0 ${pi/2} 0"
-/>
-<visual>
-    <geometry>
-        <cylinder
-            length="${lower_length}"
-            radius="${lower_radius}"
-        />
-    </geometry>
-    <origin
-        rpy="0 ${pi/2} 0"
-        xyz="${lower_length/2} 0 0"
-    />
-</visual>
-<collision>
-    <geometry>
-        <cylinder
-            length="${lower_length}"
-            radius="${lower_radius}"
-        />
-    </geometry>
-    <origin
-        rpy="0 ${pi/2} 0"
-        xyz="${lower_length/2} 0 0"
-    />
-</collision>
-</link>
-</xacro:macro>
-<xacro:link_lower_left number="1"/>
-<xacro:link_lower_left number="2"/>
-<xacro:link_lower_left number="3"/>
-<xacro:macro name="joint_elbow_to_lower_right" params="number">
-<joint name="elbow_to_lower_right_${number}" type="revolute">
-    <axis xyz="0 0 1"/>
-    <limit
-        effort="1000.0"
-        lower="${-pi/2}"
-        upper="${pi/2}"
-        velocity="0.5"
-    />
-    <origin
-        rpy="0 ${pi/2} 0"
-        xyz="0 ${-elbow_length/2} 0"
-    />
-    <parent link="elbow_${number}"/>
-    <child link="lower_right_${number}"/>
-</joint>
-</xacro:macro>
-<xacro:joint_elbow_to_lower_right number="1"/>
-<xacro:joint_elbow_to_lower_right number="2"/>
-<xacro:joint_elbow_to_lower_right number="3"/>
-<xacro:macro name="link_lower_right" params="number">
-<link name="lower_right_${number}">
-<xacro:cylinder_inertial
-    mass="${lower_mass}"
-    radius="${lower_radius}"
-    length="${lower_length}"
-    rpy="0 ${pi/2} 0"
-/>
-<visual>
-    <geometry>
-        <cylinder
-            length="${lower_length}"
-            radius="${lower_radius}"
-        />
-    </geometry>
-    <origin
-        rpy="0 ${pi/2} 0"
-        xyz="${lower_length/2} 0 0"
-    />
-</visual>
-<collision>
-    <geometry>
-        <cylinder
-            length="${lower_length}"
-            radius="${lower_radius}"
-        />
-    </geometry>
-    <origin
-        rpy="0 ${pi/2} 0"
-        xyz="${lower_length/2} 0 0"
-    />
-</collision>
-</link>
-</xacro:macro>
-<xacro:link_lower_right number="1"/>
-<xacro:link_lower_right number="2"/>
-<xacro:link_lower_right number="3"/>
-<xacro:macro name="joint_lower_left_to_lower_bot" params="number">
-<joint name="lower_left_to_lower_bot_${number}" type="revolute">
-    <axis xyz="0 0 1"/>
-    <limit
-        effort="1000.0"
-        lower="${-pi/2}"
-        upper="${pi/2}"
-        velocity="0.5"
-    />
-    <origin
-        rpy="0 0 0"
-        xyz="${lower_length} 0 0"
-    />
-    <parent link="lower_left_${number}"/>
-    <child link="lower_bot_${number}"/>
-</joint>
-</xacro:macro>
-<xacro:joint_lower_left_to_lower_bot number="1"/>
-<xacro:joint_lower_left_to_lower_bot number="2"/>
-<xacro:joint_lower_left_to_lower_bot number="3"/>
-<xacro:macro name="joint_lower_right_to_lower_bot" params="number">
-<joint name="lower_right_to_lower_bot_${number}" type="revolute">
-    <axis xyz="0 0 1"/>
-    <limit
-        effort="1000.0"
-        lower="${-pi/2}"
-        upper="${pi/2}"
-        velocity="0.5"
-    />
-    <origin
-        rpy="0 0 0"
-        xyz="${lower_length} 0 0"
-    />
-    <parent link="lower_right_${number}"/>
-    <child link="lower_bot_${number}"/>
-</joint>
-</xacro:macro>
-<gazebo>
-<xacro:joint_lower_right_to_lower_bot number="1"/>
-<xacro:joint_lower_right_to_lower_bot number="2"/>
-<xacro:joint_lower_right_to_lower_bot number="3"/>
-</gazebo>
-<xacro:macro name="link_lower_bot" params="number">
-<link name="lower_bot_${number}">
-<xacro:cylinder_inertial
-    mass="${elbow_mass}"
-    radius="${elbow_radius}"
-    length="${elbow_length}"
-    rpy="0 ${pi/2} ${pi/2}"
-/>
-<visual>
-    <geometry>
-        <cylinder
-            length="${elbow_length}"
-            radius="${elbow_radius}"
-        />
-    </geometry>
-    <origin
-        rpy="0 ${pi/2} ${pi/2}"
-        xyz="0 ${-elbow_length/2} 0"
-    />
-</visual>
-<collision>
-    <geometry>
-        <cylinder
-            length="${elbow_length}"
-            radius="${elbow_radius}"
-        />
-    </geometry>
-    <origin
-        rpy="0 ${pi/2} ${pi/2}"
-        xyz="0 ${-elbow_length/2} 0"
-    />
-</collision>
-</link>
-</xacro:macro>
-<xacro:link_lower_bot number="1"/>
-<xacro:link_lower_bot number="2"/>
-<xacro:link_lower_bot number="3"/>
-<xacro:macro name="joint_lower_bot_to_end_effector" params="number">
-<joint name="lower_bot_to_end_effector_${number}" type="revolute">
-    <axis xyz="0 1 0"/>
-    <limit
-        effort="1000.0"
-        lower="${-pi/2}"
-        upper="${pi/2}"
-        velocity="0.5"
-    />
-    <origin
-        rpy="${pi} ${pi/2} 0"
-        xyz="0 ${-elbow_length/2} 0"
-    />
-    <parent link="lower_bot_${number}"/>
-    <child link="end_effector_${number}"/>
-</joint>
-</xacro:macro>
-<xacro:joint_lower_bot_to_end_effector number="1"/>
-<xacro:joint_lower_bot_to_end_effector number="2"/>
-<xacro:joint_lower_bot_to_end_effector number="3"/>
-<xacro:macro name="link_end_effector" params="number">
-<link name="end_effector_${number}">
-<inertial>
-    <origin xyz="0 0 0" rpy="0 0 0"/>
-    <mass value="0"/>
-    <inertia ixx="0" iyy="0" izz="0" ixy="0" ixz="0" iyz="0"/>
-</inertial>
-<visual>
-    <geometry>
-        <cylinder
-            length="${end_effector_radius}"
-            radius="${end_effector_depth}"
-        />
-    </geometry>
-    <origin
-        rpy="0 ${pi/2} 0"
-        xyz="${end_effector_radius/2} 0 0"
-    />
-</visual>
-<collision>
-    <geometry>
-        <cylinder
-            length="${end_effector_radius}"
-            radius="${end_effector_depth}"
-        />
-    </geometry>
-    <origin
-        rpy="0 ${pi/2} 0"
-        xyz="${end_effector_radius/2} 0 0"
-    />
-</collision>
-</link>
-</xacro:macro>
-<xacro:link_end_effector number="1"/>
-<xacro:link_end_effector number="2"/>
-<xacro:link_end_effector number="3"/>
-<xacro:macro name="end_effector_actual">
-<link name="end_effector">
-    <visual>
-        <geometry>
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
File: model/parameters.urdf.xacro (robot description, xacro)
@@ -5,8 +5,7 @@
 <xacro:property name="upper_length" value="0.3"/>
 <xacro:property name="upper_radius" value="0.03"/>
-<xacro:property name="elbow_length" value="0.4"/>
-<xacro:property name="elbow_radius" value="0.03"/>
-<xacro:property name="lower_length" value="0.6"/>
 <xacro:property name="lower_radius" value="0.03"/>
+<xacro:property name="lower_horizontal_length" value="0.4"/>
+<xacro:property name="lower_vertical_length" value="0.6"/>
 <xacro:property name="joint_lower_limit" value="${-pi/2}"/>
 <xacro:property name="joint_upper_limit" value="${pi/2}"/>
@@ -15,6 +14,7 @@
 <xacro:property name="base_mass" value="0.1"/>
 <xacro:property name="upper_mass" value="0.04"/>
-<xacro:property name="elbow_mass" value="0.02"/>
-<xacro:property name="lower_mass" value="0.04"/>
+<xacro:property name="lower_horizontal_mass" value="0.02"/>
+<xacro:property name="lower_vertical_mass" value="0.04"/>
 <xacro:property name="end_effector_mass" value="0.05"/>
+<xacro:property name="break_indicator_radius" value="0.05"/>
 </robot>
