Commit message: Updated urdf

File: model/delta.urdf.xacro (robot description, xacro)
@@ -7,5 +7,4 @@
 <xacro:include filename="delta_upper.urdf.xacro"/>
 <xacro:include filename="delta_lower.urdf.xacro"/>
-<xacro:include filename="delta_lower_virtual.urdf.xacro"/>
 <xacro:include filename="delta_end_effector.urdf.xacro"/>
 </robot>

File: model/delta_base.urdf.xacro (robot description, xacro)
@@ -10,5 +10,5 @@
         />
     </geometry>
-    <material name="physical_link"/>
+    <material name="base"/>
 </visual>
 <collision>

File: model/delta_end_effector.urdf.xacro (robot description, xacro)
@@ -2,26 +2,20 @@
 <robot xmlns:xacro="http://www.ros.org/wiki/xacro" name="delta">
 <!-- ===== END EFFECTOR ===== -->
-<joint name="lower_bot_1_to_virtual_end_effector_offset" type="revolute">
-    <axis xyz="0 -1 0"/>
-    <limit
-        effort="1000.0"
-        lower="${-pi/2}"
-        upper="${pi/2}"
-        velocity="0.5"
+<xacro:macro name="joint_end_effector" params="number yaw">
+<joint name="lower_${number}_end_to_end_effector" type="fixed">
+    <origin rpy="0 0 0" xyz="${end_effector_radius} 0 0"/>
+    <origin
+        rpy="0 ${pi} ${yaw}"
+        xyz="${end_effector_radius} 0 0"
     />
-    <origin
-        rpy="0 0 0"
-        xyz="0 ${-lower_horizontal_length/2} 0"
-    />
-    <parent link="lower_bot_1"/>
-    <child link="virtual_end_effector_offset"/>
-</joint>
-<link name="virtual_end_effector_offset">
-</link>
-<joint name="virtual_end_effector_offset_to_end_effector" type="fixed">
-    <origin rpy="0 0 0" xyz="${end_effector_radius} 0 0"/>
-    <parent link="virtual_end_effector_offset"/>
+    <parent link="lower_${number}_end"/>
     <child link="end_effector"/>
 </joint>
+</xacro:macro>
+<xacro:joint_end_effector number="1" yaw="0"/>
+<gazebo>
+<xacro:joint_end_effector number="2" yaw="${pi*2/3}"/>
+<xacro:joint_end_effector number="3" yaw="${pi*4/3}"/>
+</gazebo>
 <link name="end_effector">
     <visual>
@@ -33,5 +27,5 @@
         </geometry>
         <origin rpy="0 0 0" xyz="0 0 0"/>
-        <material name="physical_link"/>
+        <material name="end_effector"/>
     </visual>
     <collision>

File: model/delta_lower.urdf.xacro (robot description, xacro)
@@ -2,254 +2,151 @@
 <robot xmlns:xacro="http://www.ros.org/wiki/xacro" name="delta">
 <!-- ===== LOWER TOP ===== -->
-<xacro:macro name="joint_upper_to_lower_top" params="number">
-<joint name="upper_to_lower_top_${number}" type="revolute">
+<xacro:macro name="parallel" params="parent name length width link_radius link_material">
+<joint name="${name}_alpha" type="revolute">
     <axis xyz="0 1 0"/>
-    <limit
-        effort="1000.0"
-        lower="${-pi/2}"
-        upper="${pi/2}"
-        velocity="0.5"
-    />
+    <limit effort="1000.0" lower="${-pi/2}" upper="${pi/2}" velocity="0.5"/>
     <origin
-        rpy="0 0 ${pi}"
-        xyz="${upper_length} 0 0"
-    />
-    <parent link="upper_${number}"/>
-    <child link="lower_top_${number}"/>
-</joint>
-</xacro:macro>
-<xacro:joint_upper_to_lower_top number="1"/>
-<xacro:joint_upper_to_lower_top number="2"/>
-<xacro:joint_upper_to_lower_top number="3"/>
-<xacro:macro name="link_lower_top" params="number">
-<link name="lower_top_${number}">
-<xacro:cylinder_inertial
-    mass="${lower_horizontal_mass}"
-    radius="${lower_radius}"
-    length="${lower_horizontal_length}"
-    rpy="0 ${pi/2} ${pi/2}"
-/>
-<visual>
-    <geometry>
-        <cylinder length="${lower_horizontal_length}" radius="${lower_radius}"/>
-    </geometry>
-    <origin
-        rpy="0 ${pi/2} ${pi/2}"
+        rpy="0 0 0"
         xyz="0 0 0"
     />
-    <material name="physical_link"/>
-</visual>
-<collision>
-    <geometry>
-        <cylinder length="${lower_horizontal_length}" radius="${lower_radius}"/>
-    </geometry>
-    <origin
-        rpy="0 ${pi/2} ${pi/2}"
-        xyz="0 0 0"
-    />
-</collision>
+    <parent link="${parent}"/>
+    <child link="${name}_root"/>
+</joint>
+<link name="${name}_root">
 </link>
-</xacro:macro>
-<xacro:link_lower_top number="1"/>
-<xacro:link_lower_top number="2"/>
-<xacro:link_lower_top number="3"/>
-<!-- ===== LOWER LEFT ===== -->
-<xacro:macro name="joint_lower_top_to_lower_left" params="number">
-<joint name="lower_top_to_lower_left_${number}" type="revolute">
+<joint name="${name}_L_beta_top" type="revolute">
     <axis xyz="0 0 1"/>
-    <limit
-        effort="1000.0"
-        lower="${-pi/2}"
-        upper="${pi/2}"
-        velocity="0.5"
-    />
+    <limit effort="1000.0" lower="${-pi/2}" upper="${pi/2}" velocity="0.5"/>
     <origin
         rpy="0 0 0"
-        xyz="0 ${lower_horizontal_length/2} 0"
+        xyz="0 ${width/2} 0"
     />
-    <parent link="lower_top_${number}"/>
-    <child link="lower_left_${number}"/>
+    <parent link="${name}_root"/>
+    <child link="${name}_L_link"/>
 </joint>
-</xacro:macro>
-<xacro:joint_lower_top_to_lower_left number="1"/>
-<xacro:joint_lower_top_to_lower_left number="2"/>
-<xacro:joint_lower_top_to_lower_left number="3"/>
-<xacro:macro name="link_lower_left" params="number">
-<link name="lower_left_${number}">
-<xacro:cylinder_inertial
-    mass="${lower_vertical_mass}"
-    radius="${lower_radius}"
-    length="${lower_vertical_length}"
-    rpy="0 ${pi/2} 0"
-/>
+<link name="${name}_L_link">
 <visual>
     <geometry>
         <cylinder
-            length="${lower_vertical_length}"
-            radius="${lower_radius}"
+            length="${length}"
+            radius="${link_radius}"
         />
     </geometry>
     <origin
         rpy="0 ${pi/2} 0"
-        xyz="${lower_vertical_length/2} 0 0"
+        xyz="${length/2} 0 0"
     />
-    <material name="physical_link"/>
+    <material name="${link_material}"/>
 </visual>
 <collision>
     <geometry>
         <cylinder
-            length="${lower_vertical_length}"
-            radius="${lower_radius}"
+            length="${length}"
+            radius="${link_radius}"
         />
     </geometry>
     <origin
         rpy="0 ${pi/2} 0"
-        xyz="${lower_vertical_length/2} 0 0"
+        xyz="${length/2} 0 0"
     />
 </collision>
 </link>
-</xacro:macro>
-<xacro:link_lower_left number="1"/>
-<xacro:link_lower_left number="2"/>
-<xacro:link_lower_left number="3"/>
-<!-- ===== LOWER RIGHT ===== -->
-<xacro:macro name="joint_lower_top_to_lower_right" params="number">
-<joint name="lower_top_to_lower_right_${number}" type="revolute">
+<joint name="${name}_L_beta_bot" type="revolute">
     <axis xyz="0 0 1"/>
-    <limit
-        effort="1000.0"
-        lower="${-pi/2}"
-        upper="${pi/2}"
-        velocity="0.5"
-    />
+    <limit effort="1000.0" lower="${-pi/2}" upper="${pi/2}" velocity="0.5"/>
     <origin
         rpy="0 0 0"
-        xyz="0 ${-lower_horizontal_length/2} 0"
+        xyz="${length} 0 0"
     />
-    <parent link="lower_top_${number}"/>
-    <child link="lower_right_${number}"/>
+    <parent link="${name}_L_link"/>
+    <child link="${name}_L_link_end"/>
 </joint>
-</xacro:macro>
-<xacro:joint_lower_top_to_lower_right number="1"/>
-<xacro:joint_lower_top_to_lower_right number="2"/>
-<xacro:joint_lower_top_to_lower_right number="3"/>
-<xacro:macro name="link_lower_right" params="number">
-<link name="lower_right_${number}">
-<xacro:cylinder_inertial
-    mass="${lower_vertical_mass}"
-    radius="${lower_radius}"
-    length="${lower_vertical_length}"
-    rpy="0 ${pi/2} 0"
-/>
+<link name="${name}_L_link_end">
+</link>
+<joint name="${name}_L_gamma" type="revolute">
+    <axis xyz="0 1 0"/>
+    <limit effort="1000.0" lower="${-pi/2}" upper="${pi/2}" velocity="0.5"/>
+    <origin
+        rpy="0 0 0"
+        xyz="0 ${-width/2} 0"
+    />
+    <parent link="${name}_L_link_end"/>
+    <child link="${name}_end"/>
+</joint>
+<joint name="${name}_R_beta_top" type="revolute">
+    <axis xyz="0 0 1"/>
+    <limit effort="1000.0" lower="${-pi/2}" upper="${pi/2}" velocity="0.5"/>
+    <origin
+        rpy="0 0 0"
+        xyz="0 ${-width/2} 0"
+    />
+    <parent link="${name}_root"/>
+    <child link="${name}_R_link"/>
+</joint>
+<link name="${name}_R_link">
 <visual>
     <geometry>
         <cylinder
-            length="${lower_vertical_length}"
-            radius="${lower_radius}"
+            length="${length}"
+            radius="${link_radius}"
         />
     </geometry>
     <origin
         rpy="0 ${pi/2} 0"
-        xyz="${lower_vertical_length/2} 0 0"
+        xyz="${length/2} 0 0"
     />
-    <material name="physical_link"/>
+    <material name="${link_material}"/>
 </visual>
 <collision>
     <geometry>
         <cylinder
-            length="${lower_vertical_length}"
-            radius="${lower_radius}"
+            length="${length}"
+            radius="${link_radius}"
         />
     </geometry>
     <origin
         rpy="0 ${pi/2} 0"
-        xyz="${lower_vertical_length/2} 0 0"
+        xyz="${length/2} 0 0"
     />
 </collision>
 </link>
-</xacro:macro>
-<xacro:link_lower_right number="1"/>
-<xacro:link_lower_right number="2"/>
-<xacro:link_lower_right number="3"/>
-<!-- ===== LOWER BOT ===== -->
-<xacro:macro name="joint_lower_left_to_lower_bot" params="number">
-<joint name="lower_left_to_lower_bot_${number}" type="revolute">
-    <axis xyz="0 0 -1"/>
-    <limit
-        effort="1000.0"
-        lower="${-pi/2}"
-        upper="${pi/2}"
-        velocity="0.5"
-    />
+<joint name="${name}_R_beta_bot" type="revolute">
+    <axis xyz="0 0 1"/>
+    <limit effort="1000.0" lower="${-pi/2}" upper="${pi/2}" velocity="0.5"/>
     <origin
         rpy="0 0 0"
-        xyz="${lower_vertical_length} 0 0"
+        xyz="${length} 0 0"
     />
-    <parent link="lower_left_${number}"/>
-    <child link="lower_bot_${number}"/>
+    <parent link="${name}_R_link"/>
+    <child link="${name}_R_link_end"/>
 </joint>
-</xacro:macro>
-<xacro:joint_lower_left_to_lower_bot number="1"/>
-<xacro:joint_lower_left_to_lower_bot number="2"/>
-<xacro:joint_lower_left_to_lower_bot number="3"/>
-<xacro:macro name="joint_lower_right_to_lower_bot" params="number">
-<joint name="lower_right_to_lower_bot_${number}" type="revolute">
-    <axis xyz="0 0 1"/>
-    <limit
-        effort="1000.0"
-        lower="${-pi/2}"
-        upper="${pi/2}"
-        velocity="0.5"
-    />
+<link name="${name}_R_link_end">
+</link>
+<gazebo>
+<joint name="${name}_R_gamma" type="revolute">
+    <axis xyz="0 1 0"/>
+    <limit effort="1000.0" lower="${-pi/2}" upper="${pi/2}" velocity="0.5"/>
     <origin
         rpy="0 0 0"
-        xyz="${lower_vertical_length} 0 0"
+        xyz="0 ${width/2} 0"
     />
-    <parent link="lower_right_${number}"/>
-    <child link="lower_bot_${number}"/>
+    <parent link="${name}_R_link_end"/>
+    <child link="${name}_end"/>
 </joint>
-</xacro:macro>
-<gazebo>
-<xacro:joint_lower_right_to_lower_bot number="1"/>
-<xacro:joint_lower_right_to_lower_bot number="2"/>
-<xacro:joint_lower_right_to_lower_bot number="3"/>
 </gazebo>
-<xacro:macro name="link_lower_bot" params="number">
-<link name="lower_bot_${number}">
-<xacro:cylinder_inertial
-    mass="${lower_horizontal_mass}"
-    radius="${lower_radius}"
-    length="${lower_horizontal_length}"
-    rpy="0 ${pi/2} ${pi/2}"
-/>
-<visual>
-    <geometry>
-        <cylinder
-            length="${lower_horizontal_length}"
-            radius="${lower_radius}"
-        />
-    </geometry>
-    <origin
-        rpy="0 ${pi/2} ${pi/2}"
-        xyz="0 ${-lower_horizontal_length/2} 0"
-    />
-    <material name="physical_link"/>
-</visual>
-<collision>
-    <geometry>
-        <cylinder
-            length="${lower_horizontal_length}"
-            radius="${lower_radius}"
-        />
-    </geometry>
-    <origin
-        rpy="0 ${pi/2} ${pi/2}"
-        xyz="0 ${-lower_horizontal_length/2} 0"
-    />
-</collision>
+<link name="${name}_end">
 </link>
 </xacro:macro>
-<xacro:link_lower_bot number="1"/>
-<xacro:link_lower_bot number="2"/>
-<xacro:link_lower_bot number="3"/>
+<xacro:parallel
+    parent="lower_1_parent" name="lower_1" length="${lower_length}"
+    width="${lower_width}" link_material="lower" link_radius="${lower_radius}"
+/>
+<xacro:parallel
+    parent="lower_2_parent" name="lower_2" length="${lower_length}"
+    width="${lower_width}" link_material="lower" link_radius="${lower_radius}"
+/>
+<xacro:parallel
+    parent="lower_3_parent" name="lower_3" length="${lower_length}"
+    width="${lower_width}" link_material="lower" link_radius="${lower_radius}"
+/>
 </robot>

File: model/delta_upper.urdf.xacro (robot description, xacro)
@@ -2,11 +2,11 @@
 <robot xmlns:xacro="http://www.ros.org/wiki/xacro" name="delta_parameters">
 <!-- ===== JOINTS ===== -->
-<xacro:macro name="joint_base_to_upper" params="number yaw">
-<joint name="base_to_upper_${number}" type="revolute">
+<xacro:macro name="joint_theta" params="number yaw">
+<joint name="theta_${number}" type="revolute">
     <axis xyz="0 1 0"/>
     <limit
         effort="1000.0"
-        lower="${joint_lower_limit}"
-        upper="${joint_upper_limit}"
+        lower="${-pi/2}"
+        upper="${pi/2}"
         velocity="0.5"
     />
@@ -19,7 +19,7 @@
 </joint>
 </xacro:macro>
-<xacro:joint_base_to_upper number="1" yaw="0"/>
-<xacro:joint_base_to_upper number="2" yaw="${pi*2/3}"/>
-<xacro:joint_base_to_upper number="3" yaw="${-pi*2/3}"/>
+<xacro:joint_theta number="1" yaw="0"/>
+<xacro:joint_theta number="2" yaw="${pi*2/3}"/>
+<xacro:joint_theta number="3" yaw="${-pi*2/3}"/>
 <!-- ===== LINKS ===== -->
 <xacro:macro name="link_upper" params="number">
@@ -42,5 +42,5 @@
         rpy="0 ${pi/2} 0"
     />
-    <material name="physical_link"/>
+    <material name="upper"/>
 </visual>
 <collision>
@@ -61,3 +61,19 @@
 <xacro:link_upper number="2"/>
 <xacro:link_upper number="3"/>
+<!-- ===== PARALLEL LINKAGE PARENT LINKS ===== -->
+<xacro:macro name="parallel_parent" params="parent length child">
+<joint name="${parent}_to_${child}_parent" type="fixed">
+    <origin
+        rpy="0 0 0"
+        xyz="${length} 0 0"
+    />
+    <parent link="${parent}"/>
+    <child link="${child}_parent"/>
+</joint>
+<link name="${child}_parent">
+</link>
+</xacro:macro>
+<xacro:parallel_parent parent="upper_1" length="${upper_length}" child="lower_1"/>
+<xacro:parallel_parent parent="upper_2" length="${upper_length}" child="lower_2"/>
+<xacro:parallel_parent parent="upper_3" length="${upper_length}" child="lower_3"/>
 </robot>

File: model/materials.urdf.xacro (robot description, xacro)
@@ -1,12 +1,15 @@
 <?xml version="1.0"?>
 <robot xmlns:xacro="http://www.ros.org/wiki/xacro" name="delta_materials">
-<material name="break_indicator">
-    <color rgba="1 0 0 1"/>
+<material name="base">
+    <color rgba="1 0 1 1"/>
 </material>
-<material name="physical_link">
+<material name="upper">
     <color rgba="0 1 1 1"/>
 </material>
-<material name="virtual_link">
-    <color rgba="1 0 1 0.5"/>
+<material name="lower">
+    <color rgba="0 1 0 1"/>
+</material>
+<material name="end_effector">
+    <color rgba="1 0 1 1"/>
 </material>
 </robot>

File: model/parameters.urdf.xacro (robot description, xacro)
@@ -6,8 +6,6 @@
 <xacro:property name="upper_radius" value="0.01"/>
 <xacro:property name="lower_radius" value="0.01"/>
-<xacro:property name="lower_horizontal_length" value="0.4"/>
-<xacro:property name="lower_vertical_length" value="0.6"/>
-<xacro:property name="joint_lower_limit" value="${-pi/2}"/>
-<xacro:property name="joint_upper_limit" value="${pi/2}"/>
+<xacro:property name="lower_width" value="0.4"/>
+<xacro:property name="lower_length" value="0.6"/>
 <xacro:property name="end_effector_radius" value="0.2"/>
 <xacro:property name="end_effector_depth" value="0.03"/>

Commit message: Started trying to get gazebo to work. May try making a seperate gazebo model, without the hacks necessary for urdf

File: model/delta.urdf.xacro (robot description, xacro)
@@ -8,3 +8,6 @@
 <xacro:include filename="delta_lower.urdf.xacro"/>
 <xacro:include filename="delta_end_effector.urdf.xacro"/>
+<gazebo>
+<plugin name="gazebo_ros_control" filename="libgazebo_ros_control.so"/>
+</gazebo>
 </robot>

File: model/delta_base.urdf.xacro (robot description, xacro)
@@ -1,6 +1,15 @@
 <?xml version="1.0"?>
 <robot xmlns:xacro="http://www.ros.org/wiki/xacro" name="delta_parameters">
+<link name="world"></link>
+<joint name="world_to_base" type="fixed">
+    <origin xyz="0 0 ${upper_length + lower_length + 4*end_effector_depth}" rpy="0 0 0"/>
+    <parent link="world"/>
+    <child link="base"/>
+</joint>
 <link name="base">
-<!-- root link doesn't need inertia -->
+<xacro:cylinder_inertial
+    mass="${base_mass}" radius="${base_radius}" length="${base_depth}"
+    rpy="0 0 0"
+/>
 <visual>
     <geometry>

File: model/delta_end_effector.urdf.xacro (robot description, xacro)
@@ -12,4 +12,5 @@
 </joint>
 <link name="chain_${number}_end">
+<xacro:light_inertial/>
 </link>
 </xacro:macro>
@@ -25,8 +26,6 @@
 </xacro:macro>
 <xacro:joint_chain_end_to_end_effector number="1"/>
-<gazebo>
 <xacro:joint_chain_end_to_end_effector number="2"/>
 <xacro:joint_chain_end_to_end_effector number="3"/>
-</gazebo>
 <link name="end_effector">
 <visual>

File: model/delta_lower.urdf.xacro (robot description, xacro)
@@ -2,5 +2,5 @@
 <robot xmlns:xacro="http://www.ros.org/wiki/xacro" name="delta">
 <!-- ===== LOWER TOP ===== -->
-<xacro:macro name="parallel" params="parent name length width link_radius link_material">
+<xacro:macro name="parallel" params="parent name length width link_radius link_material link_mass">
 <joint name="${name}_alpha" type="revolute">
     <axis xyz="0 1 0"/>
@@ -14,4 +14,5 @@
 </joint>
 <link name="${name}_root">
+    <xacro:light_inertial/>
 </link>
 <joint name="${name}_L_beta_top" type="revolute">
@@ -26,4 +27,10 @@
 </joint>
 <link name="${name}_L_link">
+<xacro:cylinder_inertial
+    mass="${link_mass}"
+    radius="${link_radius}"
+    length="${length}"
+    rpy="0 ${pi/2} 0"
+/>
 <visual>
     <geometry>
@@ -63,4 +70,5 @@
 </joint>
 <link name="${name}_L_link_end">
+    <xacro:light_inertial/>
 </link>
 <joint name="${name}_L_gamma" type="revolute">
@@ -85,4 +93,10 @@
 </joint>
 <link name="${name}_R_link">
+<xacro:cylinder_inertial
+    mass="${link_mass}"
+    radius="${link_radius}"
+    length="${length}"
+    rpy="0 ${pi/2} 0"
+/>
 <visual>
     <geometry>
@@ -122,6 +136,6 @@
 </joint>
 <link name="${name}_R_link_end">
+    <xacro:light_inertial/>
 </link>
-<gazebo>
 <joint name="${name}_R_gamma" type="revolute">
     <axis xyz="0 1 0"/>
@@ -134,19 +148,22 @@
     <child link="${name}_end"/>
 </joint>
-</gazebo>
 <link name="${name}_end">
+    <xacro:light_inertial/>
 </link>
 </xacro:macro>
 <xacro:parallel
     parent="lower_1_parent" name="lower_1" length="${lower_length}"
-    width="${lower_width}" link_material="lower" link_radius="${lower_radius}"
+    width="${lower_width}" link_material="lower"
+    link_radius="${lower_radius}" link_mass="${lower_mass/2}"
 />
 <xacro:parallel
     parent="lower_2_parent" name="lower_2" length="${lower_length}"
-    width="${lower_width}" link_material="lower" link_radius="${lower_radius}"
+    width="${lower_width}" link_material="lower"
+    link_radius="${lower_radius}" link_mass="${lower_mass/2}"
 />
 <xacro:parallel
     parent="lower_3_parent" name="lower_3" length="${lower_length}"
-    width="${lower_width}" link_material="lower" link_radius="${lower_radius}"
+    width="${lower_width}" link_material="lower"
+    link_radius="${lower_radius}" link_mass="${lower_mass/2}"
 />
 </robot>

File: model/delta_upper.urdf.xacro (robot description, xacro)
@@ -18,4 +18,14 @@
     <child link="upper_${number}"/>
 </joint>
+<transmission name="theta_${number}_tran">
+    <type>transmission_interface/SimpleTransmission</type>
+    <joint name="theta_${number}">
+        <hardwareInterface>hardware_interface/EffortJointInterface</hardwareInterface>
+    </joint>
+    <actuator name="theta_${number}_motor">
+        <hardwareInterface>hardware_interface/EffortJointInterface</hardwareInterface>
+        <mechanicalReduction>1</mechanicalReduction>
+    </actuator>
+</transmission>
 </xacro:macro>
 <xacro:joint_theta number="1" yaw="0"/>
@@ -97,4 +107,5 @@
 </joint>
 <link name="${child}_parent">
+    <xacro:light_inertial/>
 </link>
 </xacro:macro>

File: model/inertia.urdf.xacro (robot description, xacro)
@@ -15,3 +15,15 @@
 </inertial>
 </xacro:macro>
+<!-- Not allowed to have links with zero mass, so put an inertial
+element with very low mass and inertia
+Should replace the two revolute joints + virtual link, with
+a revolute2 joint for gazebo
+-->
+<xacro:macro name="light_inertial">
+<inertial>
+    <origin rpy="0 0 0" xyz="0 0 0"/>
+    <mass value="0.1"/>
+    <inertia ixx="0.001" iyy="0.001" izz="0.001" ixy="0" ixz="0" iyz="0"/>
+</inertial>
+</xacro:macro>
 </robot>

File: model/parameters.urdf.xacro (robot description, xacro)
@@ -12,6 +12,5 @@
 <xacro:property name="base_mass" value="0.1"/>
 <xacro:property name="upper_mass" value="0.04"/>
-<xacro:property name="lower_horizontal_mass" value="0.02"/>
-<xacro:property name="lower_vertical_mass" value="0.04"/>
+<xacro:property name="lower_mass" value="0.06"/>
 <xacro:property name="end_effector_mass" value="0.05"/>
 <xacro:property name="break_indicator_radius" value="0.03"/>
