Commit message: ROS urdf working in new format

File: model/delta/gazebo.urdf.xacro (robot description, xacro)
@@ -8,6 +8,4 @@
 <xacro:include filename="delta_lower.urdf.xacro"/>
 <xacro:include filename="delta_end_effector.urdf.xacro"/>
-<gazebo>
 <plugin name="gazebo_ros_control" filename="libgazebo_ros_control.so"/>
-</gazebo>
 </robot>

File: model/delta/links/base.urdf.xacro (robot description, xacro)
@@ -1,4 +1,4 @@
 <?xml version="1.0"?>
-<robot xmlns:xacro="http://www.ros.org/wiki/xacro" name="delta_parameters">
+<robot xmlns:xacro="http://www.ros.org/wiki/xacro" name="base">
 <link name="world"></link>
 <joint name="world_to_base" type="fixed">

File: model/delta/links/end_effector.urdf.xacro (robot description, xacro)
@@ -1,31 +1,4 @@
 <?xml version="1.0"?>
 <robot xmlns:xacro="http://www.ros.org/wiki/xacro" name="delta">
-<!-- ===== END EFFECTOR ===== -->
-<xacro:macro name="chain_end" params="number yaw">
-<joint name="lower_end_to_chain_end_${number}" type="fixed">
-    <origin
-        rpy="0 ${pi} ${yaw}"
-        xyz="${end_effector_radius} 0 0"
-    />
-    <parent link="lower_${number}_end"/>
-    <child link="chain_${number}_end"/>
-</joint>
-<link name="chain_${number}_end">
-<xacro:light_inertial/>
-</link>
-</xacro:macro>
-<xacro:chain_end number="1" yaw="0"/>
-<xacro:chain_end number="2" yaw="${pi*2/3}"/>
-<xacro:chain_end number="3" yaw="${pi*4/3}"/>
-<xacro:macro name="joint_chain_end_to_end_effector" params="number">
-<joint name="chain_${number}_end_to_end_effector" type="fixed">
-    <origin xyz="0 0 0" rpy="0 0 0"/>
-    <parent link="chain_${number}_end"/>
-    <child link="end_effector"/>
-</joint>
-</xacro:macro>
-<xacro:joint_chain_end_to_end_effector number="1"/>
-<xacro:joint_chain_end_to_end_effector number="2"/>
-<xacro:joint_chain_end_to_end_effector number="3"/>
 <link name="end_effector">
 <visual>

File: model/delta/ros_joints/upper.urdf.xacro (robot description, xacro)
@@ -1,5 +1,5 @@
 <?xml version="1.0"?>
 <robot xmlns:xacro="http://www.ros.org/wiki/xacro" name="delta_parameters">
-<!-- ===== JOINTS ===== -->
+<!-- ===== THETA ===== -->
 <xacro:macro name="joint_theta" params="number yaw">
 <joint name="theta_${number}" type="revolute">
@@ -32,69 +32,6 @@
 <xacro:joint_theta number="2" yaw="${pi*2/3}"/>
 <xacro:joint_theta number="3" yaw="${-pi*2/3}"/>
-<!-- ===== LINKS ===== -->
-<xacro:macro name="link_upper" params="number">
-<link name="upper_${number}">
-<xacro:cylinder_inertial
-    mass="${upper_mass}"
-    radius="${upper_radius}"
-    length="${upper_length}"
-    rpy="0 ${pi/2} 0"
-/>
-<visual>
-    <geometry>
-        <cylinder
-            length="${upper_length}"
-            radius="${upper_radius}"
-        />
-    </geometry>
-    <origin
-        xyz="${upper_length/2} 0 0"
-        rpy="0 ${pi/2} 0"
-    />
-    <material name="upper"/>
-</visual>
-<collision>
-    <geometry>
-        <cylinder
-            length="${upper_length}"
-            radius="${upper_radius}"
-        />
-    </geometry>
-    <origin
-        xyz="${upper_length/2} 0 0"
-        rpy="0 ${pi/2} 0"
-    />
-</collision>
-<visual>
-    <geometry>
-        <cylinder
-            length="${lower_width}"
-            radius="${upper_radius}"
-        />
-    </geometry>
-    <origin
-        xyz="${upper_length} 0 0"
-        rpy="${pi/2} 0 0"
-    />
-    <material name="upper"/>
-</visual>
-<collision>
-    <geometry>
-        <cylinder
-            length="${lower_width}"
-            radius="${upper_radius}"
-        />
-    </geometry>
-    <origin
-        xyz="${upper_length} 0 0"
-        rpy="${pi/2} 0 0"
-    />
-</collision>
-</link>
-</xacro:macro>
-<xacro:link_upper number="1"/>
-<xacro:link_upper number="2"/>
-<xacro:link_upper number="3"/>
-<!-- ===== PARALLEL LINKAGE PARENT LINKS ===== -->
+<!-- ===== JOINT AND VIRTUAL LINK FOR ROOT OF
+           LOWER PARALLEL LINKAGE             ===== -->
 <xacro:macro name="parallel_parent" params="parent length child">
 <joint name="${parent}_to_${child}_parent" type="fixed">
@@ -107,5 +44,4 @@
 </joint>
 <link name="${child}_parent">
-    <xacro:light_inertial/>
 </link>
 </xacro:macro>

File: model/macros/inertia.urdf.xacro (robot description, xacro)
@@ -15,15 +15,3 @@
 </inertial>
 </xacro:macro>
-<!-- Not allowed to have links with zero mass, so put an inertial
-element with very low mass and inertia
-Should replace the two revolute joints + virtual link, with
-a revolute2 joint for gazebo
--->
-<xacro:macro name="light_inertial">
-<inertial>
-    <origin rpy="0 0 0" xyz="0 0 0"/>
-    <mass value="0.1"/>
-    <inertia ixx="0.001" iyy="0.001" izz="0.001" ixy="0" ixz="0" iyz="0"/>
-</inertial>
-</xacro:macro>
 </robot>
