Commit message: More work on gazebo model

File: model/delta/gazebo.sdf.xacro (robot description, xacro)
@@ -1,14 +1,16 @@
 <?xml version="1.0"?>
-<model xmlns:xacro="http://www.ros.org/wiki/xacro">
-<name>delta</name>
-<xacro:include filename="parameters.urdf.xacro"/>
-<xacro:include filename="materials.urdf.xacro"/>
-<xacro:include filename="../macros/inertia.urdf.xacro"/>
-<xacro:include filename="links/base.urdf.xacro"/>
+<sdf xmlns:xacro="http://www.ros.org/wiki/xacro" version='1.4'>
+<model name="delta">
+<static>false</static>
+<xacro:include filename="parameters.xacro"/>
+<xacro:include filename="../macros/inertia.xacro"/>
+<xacro:include filename="gazebo_links/base.sdf.xacro"/>
+<xacro:include filename="gazebo_links/upper.sdf.xacro"/>
 <!--
-<xacro:include filename="links/upper.urdf.xacro"/>
-<xacro:include filename="links/lower.urdf.xacro"/>
-<xacro:include filename="links/end_effector.urdf.xacro"/>
+<xacro:include filename="gazebo_links/lower.sdf.xacro"/>
+<xacro:include filename="gazebo_links/end_effector.sdf.xacro"/>
+-->
 <xacro:include filename="gazebo_joints/upper.urdf.xacro"/>
+<!--
 <xacro:include filename="gazebo_joints/lower.urdf.xacro"/>
 <xacro:include filename="gazebo_joints/end_effector.urdf.xacro"/>
@@ -16,2 +18,3 @@
 -->
 </model>
+</sdf>

File: model/delta/gazebo_joints/upper.urdf.xacro (robot description, xacro)
@@ -4,28 +4,12 @@
 <xacro:macro name="joint_theta" params="number yaw">
 <joint name="theta_${number}" type="revolute">
-    <axis xyz="0 1 0"/>
-    <limit
-        effort="1000.0"
-        lower="${-pi/2}"
-        upper="${pi/2}"
-        velocity="0.5"
-    />
-    <origin
-        rpy="0 0 ${yaw}"
-        xyz="${cos(yaw)*base_radius} ${sin(yaw)*base_radius} 0"
-    />
-    <parent link="base"/>
-    <child link="upper_${number}"/>
+    <axis><xyz>0 1 0</xyz></axis>
+    <pose>
+        0 0 ${yaw}
+        ${cos(yaw)*base_radius} ${sin(yaw)*base_radius} 0
+    </pose>
+    <parent>base</parent>
+    <child>upper_${number}</child>
 </joint>
-<transmission name="theta_${number}_tran">
-    <type>transmission_interface/SimpleTransmission</type>
-    <joint name="theta_${number}">
-        <hardwareInterface>hardware_interface/EffortJointInterface</hardwareInterface>
-    </joint>
-    <actuator name="theta_${number}_motor">
-        <hardwareInterface>hardware_interface/EffortJointInterface</hardwareInterface>
-        <mechanicalReduction>1</mechanicalReduction>
-    </actuator>
-</transmission>
 </xacro:macro>
 <xacro:joint_theta number="1" yaw="0"/>

File: model/delta/ros.urdf.xacro (robot description, xacro)
@@ -1,11 +1,10 @@
 <?xml version="1.0"?>
 <robot xmlns:xacro="http://www.ros.org/wiki/xacro" name="delta">
-<xacro:include filename="parameters.urdf.xacro"/>
+<xacro:include filename="parameters.xacro"/>
 <xacro:include filename="materials.urdf.xacro"/>
-<xacro:include filename="../macros/inertia.urdf.xacro"/>
-<xacro:include filename="links/base.urdf.xacro"/>
-<xacro:include filename="links/upper.urdf.xacro"/>
-<xacro:include filename="links/lower.urdf.xacro"/>
-<xacro:include filename="links/end_effector.urdf.xacro"/>
+<xacro:include filename="ros_links/base.urdf.xacro"/>
+<xacro:include filename="ros_links/upper.urdf.xacro"/>
+<xacro:include filename="ros_links/lower.urdf.xacro"/>
+<xacro:include filename="ros_links/end_effector.urdf.xacro"/>
 <xacro:include filename="ros_joints/upper.urdf.xacro"/>
 <xacro:include filename="ros_joints/lower.urdf.xacro"/>

File: model/delta/ros_joints/upper.urdf.xacro (robot description, xacro)
@@ -1,4 +1,4 @@
 <?xml version="1.0"?>
-<robot xmlns:xacro="http://www.ros.org/wiki/xacro" name="delta_parameters">
+<robot xmlns:xacro="http://www.ros.org/wiki/xacro">
 <!-- ===== THETA ===== -->
 <xacro:macro name="joint_theta" params="number yaw">

File: model/delta/ros_links/base.urdf.xacro (robot description, xacro)
@@ -8,8 +8,4 @@
 </joint>
 <link name="base">
-<xacro:cylinder_inertial
-    mass="${base_mass}" radius="${base_radius}" length="${base_depth}"
-    rpy="0 0 0"
-/>
 <visual>
     <geometry>

File: model/delta/ros_links/upper.urdf.xacro (robot description, xacro)
@@ -3,10 +3,4 @@
 <xacro:macro name="link_upper" params="number">
 <link name="upper_${number}">
-<xacro:cylinder_inertial
-    mass="${upper_mass}"
-    radius="${upper_radius}"
-    length="${upper_length}"
-    rpy="0 ${pi/2} 0"
-/>
 <visual>
     <geometry>

Commit message: Getting gazebo model working

File: model/delta/gazebo.sdf.xacro (robot description, xacro)
@@ -1,4 +1,4 @@
-<?xml version="1.0"?>
-<sdf xmlns:xacro="http://www.ros.org/wiki/xacro" version='1.4'>
+<?xml version='1.0'?>
+<sdf version='1.4' xmlns:xacro="http://www.ros.org/wiki/xacro">
 <model name="delta">
 <static>false</static>
@@ -7,14 +7,15 @@
 <xacro:include filename="gazebo_links/base.sdf.xacro"/>
 <xacro:include filename="gazebo_links/upper.sdf.xacro"/>
+<xacro:include filename="gazebo_links/lower.sdf.xacro"/>
 <!--
-<xacro:include filename="gazebo_links/lower.sdf.xacro"/>
 <xacro:include filename="gazebo_links/end_effector.sdf.xacro"/>
 -->
-<xacro:include filename="gazebo_joints/upper.urdf.xacro"/>
+<xacro:include filename="gazebo_joints/upper.sdf.xacro"/>
+<xacro:include filename="gazebo_joints/lower.sdf.xacro"/>
 <!--
-<xacro:include filename="gazebo_joints/lower.urdf.xacro"/>
 <xacro:include filename="gazebo_joints/end_effector.urdf.xacro"/>
 <plugin name="gazebo_ros_control" filename="libgazebo_ros_control.so"/>
 -->
+<plugin name="gazebo_ros_control" filename="libgazebo_ros_control.so"/>
 </model>
 </sdf>

File: model/delta/gazebo_links/base.sdf.xacro (robot description, xacro)
@@ -1,15 +1,22 @@
 <?xml version="1.0"?>
-<robot xmlns:xacro="http://www.ros.org/wiki/xacro" name="base">
-<link name="world">
-</link>
-<joint name="world_to_base" type="fixed">
-    <pose>
-        0 0 ${upper_length + lower_length + 4*end_effector_depth}
-        0 0 0
-    </pose>
-    <parent>world</parent>
-    <child>base</child>
-</joint>
+<sdf xmlns:xacro="http://www.ros.org/wiki/xacro" name="base">
 <link name="base">
+<pose> 0 0 0 0 0 0</pose>
+<visual name="base_visual">
+    <geometry>
+        <cylinder>
+            <length>${base_depth}</length>
+            <radius>${base_radius}</radius>
+        </cylinder>
+    </geometry>
+</visual>
+<collision name="base_collision">
+    <geometry>
+        <cylinder>
+            <length>${base_depth}</length>
+            <radius>${base_radius}</radius>
+        </cylinder>
+    </geometry>
+</collision>
 <inertial>
     <mass>${base_mass}</mass>
@@ -20,20 +27,4 @@
     />
 </inertial>
-<visual name="visual">
-    <geometry>
-        <cylinder>
-            <length>${base_depth}</length>
-            <radius>${base_radius}</radius>
-        </cylinder>
-    </geometry>
-</visual>
-<collision name="collision">
-    <geometry>
-        <cylinder>
-            <length>${base_depth}</length>
-            <radius>${base_radius}</radius>
-        </cylinder>
-    </geometry>
-</collision>
 </link>
-</robot>
+</sdf>

File: model/delta/gazebo_links/lower.sdf.xacro (robot description, xacro)
@@ -2,74 +2,90 @@
 <robot xmlns:xacro="http://www.ros.org/wiki/xacro" name="delta">
 <!-- ===== LOWER TOP ===== -->
-<xacro:macro name="link_lower" params="number">
+<xacro:macro name="link_lower" params="number yaw">
 <link name="lower_${number}_L_link">
-<xacro:cylinder_inertial
-    mass="${lower_mass}"
-    radius="${lower_radius}"
-    length="${lower_length}"
-    rpy="0 ${pi/2} 0"
-/>
-<visual>
+<pose>
+    ${(base_radius + upper_length)*cos(yaw) - (lower_width/2)*sin(yaw)}
+    ${(base_radius + upper_length)*sin(yaw) + (lower_width/2)*cos(yaw)}
+    0
+    0 0 ${yaw}
+</pose>
+<visual name="lower_${number}_L_link_visual">
+    <pose>
+        ${lower_length/2} 0 0
+        0 ${pi/2} 0
+    </pose>
     <geometry>
-        <cylinder
-            length="${lower_length}"
-            radius="${lower_radius}"
-        />
+        <cylinder>
+            <length>${lower_length}</length>
+            <radius>${lower_radius}</radius>
+        </cylinder>
     </geometry>
-    <origin
-        rpy="0 ${pi/2} 0"
-        xyz="${lower_length/2} 0 0"
+</visual>
+<collision name="lower_${number}_L_link_collision">
+    <pose>
+        ${lower_length/2} 0 0
+        0 ${pi/2} 0
+    </pose>
+    <geometry>
+        <cylinder>
+            <length>${lower_length}</length>
+            <radius>${lower_radius}</radius>
+        </cylinder>
+    </geometry>
+</collision>
+<inertial>
+    <mass>${lower_mass}</mass>
+    <pose>${lower_length/2} 0 0 0 ${pi/2} 0</pose>
+    <xacro:cylinder_inertia_sdf
+        mass="${lower_mass}"
+        radius="${lower_radius}"
+        length="${lower_length}"
     />
-    <material name="lower"/>
-</visual>
-<collision>
-    <geometry>
-        <cylinder
-            length="${lower_length}"
-            radius="${lower_radius}"
-        />
-    </geometry>
-    <origin
-        rpy="0 ${pi/2} 0"
-        xyz="${lower_length/2} 0 0"
-    />
-</collision>
+</inertial>
 </link>
 <link name="lower_${number}_R_link">
-<xacro:cylinder_inertial
-    mass="${lower_mass}"
-    radius="${lower_radius}"
-    length="${lower_length}"
-    rpy="0 ${pi/2} 0"
-/>
-<visual>
+<pose>
+    ${(base_radius + upper_length)*cos(yaw) + (lower_width/2)*sin(yaw)}
+    ${(base_radius + upper_length)*sin(yaw) - (lower_width/2)*cos(yaw)}
+    0
+    0 0 ${yaw}
+</pose>
+<visual name="lower_${number}_R_link_visual">
+    <pose>
+        ${lower_length/2} 0 0
+        0 ${pi/2} 0
+    </pose>
     <geometry>
-        <cylinder
-            length="${lower_length}"
-            radius="${lower_radius}"
-        />
+        <cylinder>
+            <length>${lower_length}</length>
+            <radius>${lower_radius}</radius>
+        </cylinder>
     </geometry>
-    <origin
-        rpy="0 ${pi/2} 0"
-        xyz="${lower_length/2} 0 0"
+</visual>
+<collision name="lower_${number}_R_link_collision">
+    <pose>
+        ${lower_length/2} 0 0
+        0 ${pi/2} 0
+    </pose>
+    <geometry>
+        <cylinder>
+            <length>${lower_length}</length>
+            <radius>${lower_radius}</radius>
+        </cylinder>
+    </geometry>
+</collision>
+<inertial>
+    <mass>${lower_mass}</mass>
+    <pose>${lower_length/2} 0 0 0 ${pi/2} 0</pose>
+    <xacro:cylinder_inertia_sdf
+        mass="${lower_mass}"
+        radius="${lower_radius}"
+        length="${lower_length}"
     />
-    <material name="lower"/>
-</visual>
-<collision>
-    <geometry>
-        <cylinder
-            length="${lower_length}"
-            radius="${lower_radius}"
-        />
-    </geometry>
-    <origin
-        rpy="0 ${pi/2} 0"
-        xyz="${lower_length/2} 0 0"
-    />
-</collision>
+</inertial>
 </link>
 </xacro:macro>
-<xacro:link_lower number="1"/>
-<xacro:link_lower number="2"/>
-<xacro:link_lower number="3"/>
+<xacro:link_lower number="1" yaw="0"/>
+<xacro:link_lower number="2" yaw="${2*pi/3}"/>
+<xacro:link_lower number="3" yaw="${-2*pi/3}"/>
 </robot>

File: model/delta/gazebo_links/upper.sdf.xacro (robot description, xacro)
@@ -1,9 +1,61 @@
 <?xml version="1.0"?>
 <robot xmlns:xacro="http://www.ros.org/wiki/xacro" name="delta_parameters">
-<xacro:macro name="link_upper" params="number">
+<xacro:macro name="link_upper" params="number yaw">
 <link name="upper_${number}">
+<pose>
+    ${base_radius*cos(yaw)} ${base_radius*sin(yaw)} 0
+    0 0 ${yaw}
+</pose>
+<visual name="upper_${number}_visual">
+    <pose>
+        ${upper_length/2} 0 0
+        0 ${pi/2} 0
+    </pose>
+    <geometry>
+        <cylinder>
+            <length>${upper_length}</length>
+            <radius>${upper_radius}</radius>
+        </cylinder>
+    </geometry>
+</visual>
+<collision name="upper_${number}_collision">
+    <pose>
+        ${upper_length/2} 0 0
+        0 ${pi/2} 0
+    </pose>
+    <geometry>
+        <cylinder>
+            <length>${upper_length}</length>
+            <radius>${upper_radius}</radius>
+        </cylinder>
+    </geometry>
+</collision>
+<visual name="upper_${number}_visual2">
+    <pose>
+        ${upper_length} 0 0
+        ${pi/2} 0 0
+    </pose>
+    <geometry>
+        <cylinder>
+            <length>${lower_width}</length>
+            <radius>${upper_radius}</radius>
+        </cylinder>
+    </geometry>
+</visual>
+<collision name="upper_${number}_collision2">
+    <pose>
+        ${upper_length} 0 0
+        ${pi/2} 0 0
+    </pose>
+    <geometry>
+        <cylinder>
+            <length>${lower_width}</length>
+            <radius>${upper_radius}</radius>
+        </cylinder>
+    </geometry>
+</collision>
 <inertial>
     <mass>${upper_mass}</mass>
-    <pose>0 0 0 0 ${pi/2} 0</pose>
+    <pose>0 0 ${upper_length/2} 0 0 0</pose>
     <xacro:cylinder_inertia_sdf
         mass="${upper_mass}"
@@ -12,56 +64,8 @@
     />
 </inertial>
-<visual name="visual">
-    <geometry>
-        <cylinder>
-            <length>${upper_length}</length>
-            <radius>${upper_radius}</radius>
-        </cylinder>
-    </geometry>
-    <pose>
-        ${upper_length/2} 0 0
-        0 ${pi/2} 0
-    </pose>
-</visual>
-<collision name="collision">
-    <geometry>
-        <cylinder>
-            <length>${upper_length}</length>
-            <radius>${upper_radius}</radius>
-        </cylinder>
-    </geometry>
-    <pose>
-        ${upper_length/2} 0 0
-        0 ${pi/2} 0
-    </pose>
-</collision>
-<visual name="visual">
-    <geometry>
-        <cylinder>
-            <length>${lower_width}</length>
-            <radius>${upper_radius}</radius>
-        </cylinder>
-    </geometry>
-    <pose>
-        ${upper_length} 0 0
-        ${pi/2} 0 0
-    </pose>
-</visual>
-<collision name="collision">
-    <geometry>
-        <cylinder>
-            length="${lower_width}"
-            radius="${upper_radius}"
-        </cylinder>
-    </geometry>
-    <pose>
-        ${upper_length} 0 0
-        ${pi/2} 0 0
-    </pose>
-</collision>
 </link>
 </xacro:macro>
-<xacro:link_upper number="1"/>
-<xacro:link_upper number="2"/>
-<xacro:link_upper number="3"/>
+<xacro:link_upper number="1" yaw="0"/>
+<xacro:link_upper number="2" yaw="${2*pi/3}"/>
+<xacro:link_upper number="3" yaw="${-2*pi/3}"/>
 </robot>

File: model/delta/parameters.xacro (robot description, xacro)
@@ -2,5 +2,5 @@
 <robot xmlns:xacro="http://www.ros.org/wiki/xacro" name="delta_parameters">
 <xacro:property name="base_radius" value="0.3"/>
-<xacro:property name="base_depth" value="0.02"/>
+<xacro:property name="base_depth" value="0.05"/>
 <xacro:property name="upper_length" value="0.3"/>
 <xacro:property name="upper_radius" value="0.01"/>

File: model/delta/ros_joints/upper.urdf.xacro (robot description, xacro)
@@ -18,4 +18,14 @@
     <child link="upper_${number}"/>
 </joint>
+<transmission name="theta_${number}_tran">
+    <type>transmission_interface/SimpleTransmission</type>
+    <joint name="theta_${number}">
+        <hardwareInterface>EffortJointInterface</hardwareInterface>
+    </joint>
+    <actuator name="theta_${number}">
+        <hardwareInterface>EffortJointInterface</hardwareInterface>
+        <mechanicalReduction>1</mechanicalReduction>
+    </actuator>
+</transmission>
 </xacro:macro>
 <xacro:joint_theta number="1" yaw="0"/>
