Commit message: Gazebo model working

File: model/delta/gazebo.sdf.xacro (robot description, xacro)
@@ -8,13 +8,8 @@
 <xacro:include filename="gazebo_links/upper.sdf.xacro"/>
 <xacro:include filename="gazebo_links/lower.sdf.xacro"/>
-<!--
 <xacro:include filename="gazebo_links/end_effector.sdf.xacro"/>
--->
 <xacro:include filename="gazebo_joints/upper.sdf.xacro"/>
 <xacro:include filename="gazebo_joints/lower.sdf.xacro"/>
-<!--
-<xacro:include filename="gazebo_joints/end_effector.urdf.xacro"/>
-<plugin name="gazebo_ros_control" filename="libgazebo_ros_control.so"/>
--->
+<xacro:include filename="gazebo_joints/end_effector.sdf.xacro"/>
 <plugin name="gazebo_ros_control" filename="libgazebo_ros_control.so"/>
 </model>

File: model/delta/gazebo_joints/end_effector.sdf.xacro (robot description, xacro)
@@ -1,19 +1,28 @@
 <?xml version="1.0"?>
 <robot xmlns:xacro="http://www.ros.org/wiki/xacro" name="delta">
-<xacro:macro name="joints_end_effector" params="number">
-<joint name="lower_L_to_end_effector_${number}" type="fixed">
-    <origin
-        xyz="${end_effector_radius} ${-lower_width/2} 0"
-        rpy="0 ${pi} ${-number * pi * 2/3}"/>
-    <parent link="lower_${number}_L_end"/>
-    <child link="end_effector"/>
+<xacro:macro name="joints_end_effector" params="number yaw">
+<joint name="lower_${number}_L_ball_bot" type="ball">
+    <pose>
+        ${end_effector_radius*cos(yaw) - (lower_width/2)*sin(yaw)}
+        ${end_effector_radius*sin(yaw) + (lower_width/2)*cos(yaw)}
+        0
+        0 0 ${yaw}
+    </pose>
+    <parent>lower_${number}_L_link</parent>
+    <child>end_effector</child>
 </joint>
-<joint name="lower_R_to_end_effector_${number}" type="fixed">
-    <origin
-        xyz="${end_effector_radius} ${lower_width/2} 0"
-        rpy="0 ${pi} ${-number * pi * 2/3}"/>
-    <parent link="lower_${number}_L_end"/>
-    <child link="end_effector"/>
+<joint name="lower_${number}_R_ball_bot" type="ball">
+    <pose>
+        ${end_effector_radius*cos(yaw) + (lower_width/2)*sin(yaw)}
+        ${end_effector_radius*sin(yaw) - (lower_width/2)*cos(yaw)}
+        0
+        0 0 ${yaw}
+    </pose>
+    <parent>lower_${number}_R_link</parent>
+    <child>end_effector</child>
 </joint>
 </xacro:macro>
+<xacro:joints_end_effector number="1" yaw="0"/>
+<xacro:joints_end_effector number="2" yaw="${2*pi/3}"/>
+<xacro:joints_end_effector number="3" yaw="${-2*pi/3}"/>
 </robot>

File: model/delta/gazebo_links/base.sdf.xacro (robot description, xacro)
@@ -2,5 +2,5 @@
 <sdf xmlns:xacro="http://www.ros.org/wiki/xacro" name="base">
 <link name="base">
-<pose> 0 0 0 0 0 0</pose>
+<pose> 0 0 ${base_height} 0 0 0</pose>
 <visual name="base_visual">
     <geometry>

File: model/delta/gazebo_links/end_effector.sdf.xacro (robot description, xacro)
@@ -1,63 +1,65 @@
 <?xml version="1.0"?>
 <robot xmlns:xacro="http://www.ros.org/wiki/xacro" name="delta">
+<xacro:macro name="end_effector_attachment" params="number yaw">
+<visual name="end_effector_attachment_${number}_visual">
+    <pose>
+        ${end_effector_radius*cos(yaw)}
+        ${end_effector_radius*sin(yaw)}
+        0
+        0 ${pi/2} ${yaw + pi/2}
+    </pose>
+    <geometry>
+        <cylinder>
+            <length>${lower_width}</length>
+            <radius>${end_effector_depth/2}</radius>
+        </cylinder>
+    </geometry>
+</visual>
+<collision name="end_effector_attachment_${number}_collision">
+    <pose>
+        ${end_effector_radius*cos(yaw)}
+        ${end_effector_radius*sin(yaw)}
+        0
+        0 ${pi/2} ${yaw + pi/2}
+    </pose>
+    <geometry>
+        <cylinder>
+            <length>${lower_width}</length>
+            <radius>${end_effector_depth/2}</radius>
+        </cylinder>
+    </geometry>
+</collision>
+</xacro:macro>
 <link name="end_effector">
-<visual>
+<pose> 0 0 0 0 0 0</pose>
+<visual name="end_effector_visual">
+    <pose>0 0 0 0 0 0</pose>
     <geometry>
-        <cylinder
-            length="${end_effector_depth}"
-            radius="${end_effector_radius}"
-        />
+        <cylinder>
+            <length>${end_effector_depth}</length>
+            <radius>${end_effector_radius}</radius>
+        </cylinder>
     </geometry>
-    <origin rpy="0 0 0" xyz="0 0 0"/>
-    <material name="end_effector"/>
 </visual>
-<collision>
+<collision name="end_effector_collision">
+    <pose>0 0 0 0 0 0</pose>
     <geometry>
-        <cylinder
-            length="${end_effector_depth}"
-            radius="${end_effector_radius}"
-        />
+        <cylinder>
+            <length>${end_effector_depth}</length>
+            <radius>${end_effector_radius}</radius>
+        </cylinder>
     </geometry>
-    <origin rpy="0 0 0" xyz="0 0 0"/>
 </collision>
-<visual>
-    <geometry>
-        <cylinder length="${lower_width}" radius="${end_effector_depth/2}" />
-    </geometry>
-    <origin xyz="${end_effector_radius} 0 0" rpy="0 ${pi/2} ${pi/2}" />
-    <material name="end_effector"/>
-</visual>
-<collision>
-    <geometry>
-        <cylinder length="${lower_width}" radius="${end_effector_depth/2}" />
-    </geometry>
-    <origin xyz="${end_effector_radius} 0 0" rpy="0 ${pi/2} ${pi/2}" />
-</collision>
-<visual>
-    <geometry>
-        <cylinder length="${lower_width}" radius="${end_effector_depth/2}" />
-    </geometry>
-    <origin xyz="${cos(pi*2/3)*end_effector_radius} ${sin(pi*2/3)*end_effector_radius} 0" rpy="0 ${pi/2} ${pi*7/6}" />
-    <material name="end_effector"/>
-</visual>
-<collision>
-    <geometry>
-        <cylinder length="${lower_width}" radius="${end_effector_depth/2}" />
-    </geometry>
-    <origin xyz="${cos(pi*2/3)*end_effector_radius} ${sin(pi*2/3)*end_effector_radius} 0" rpy="0 ${pi/2} ${pi*7/6}" />
-</collision>
-<visual>
-    <geometry>
-        <cylinder length="${lower_width}" radius="${end_effector_depth/2}" />
-    </geometry>
-    <origin xyz="${cos(pi*4/3)*end_effector_radius} ${sin(pi*4/3)*end_effector_radius} 0" rpy="0 ${pi/2} ${pi*11/6}" />
-    <material name="end_effector"/>
-</visual>
-<collision>
-    <geometry>
-        <cylinder length="${lower_width}" radius="${end_effector_depth/2}" />
-    </geometry>
-    <origin xyz="${cos(pi*4/3)*end_effector_radius} ${sin(pi*4/3)*end_effector_radius} 0" rpy="0 ${pi/2} ${pi*11/6}" />
-</collision>
+<xacro:end_effector_attachment number="1" yaw="0"/>
+<xacro:end_effector_attachment number="2" yaw="${2*pi/3}"/>
+<xacro:end_effector_attachment number="3" yaw="${-2*pi/3}"/>
+<inertial>
+    <mass>${end_effector_mass}</mass>
+    <xacro:cylinder_inertia_sdf
+        mass="${end_effector_mass}"
+        radius="${end_effector_radius}"
+        length="${end_effector_depth}"
+    />
+</inertial>
 </link>
 </robot>

File: model/delta/gazebo_links/lower.sdf.xacro (robot description, xacro)
@@ -7,6 +7,6 @@
     ${(base_radius + upper_length)*cos(yaw) - (lower_width/2)*sin(yaw)}
     ${(base_radius + upper_length)*sin(yaw) + (lower_width/2)*cos(yaw)}
-    0
-    0 0 ${yaw}
+    ${base_height}
+    0 ${pi - lower_inclination} ${yaw}
 </pose>
 <visual name="lower_${number}_L_link_visual">
@@ -48,6 +48,6 @@
     ${(base_radius + upper_length)*cos(yaw) + (lower_width/2)*sin(yaw)}
     ${(base_radius + upper_length)*sin(yaw) - (lower_width/2)*cos(yaw)}
-    0
-    0 0 ${yaw}
+    ${base_height}
+    0 ${pi - lower_inclination} ${yaw}
 </pose>
 <visual name="lower_${number}_R_link_visual">

File: model/delta/gazebo_links/upper.sdf.xacro (robot description, xacro)
@@ -4,5 +4,5 @@
 <link name="upper_${number}">
 <pose>
-    ${base_radius*cos(yaw)} ${base_radius*sin(yaw)} 0
+    ${base_radius*cos(yaw)} ${base_radius*sin(yaw)} ${base_height}
     0 0 ${yaw}
 </pose>
@@ -57,5 +57,14 @@
 <inertial>
     <mass>${upper_mass}</mass>
-    <pose>0 0 ${upper_length/2} 0 0 0</pose>
+    <pose>${upper_length/2} 0 0 0 ${pi/2} 0</pose>
+    <xacro:cylinder_inertia_sdf
+        mass="${upper_mass}"
+        radius="${upper_radius}"
+        length="${upper_length}"
+    />
+</inertial>
+<inertial>
+    <mass>${upper_mass}</mass>
+    <pose>${upper_length} 0 0 ${pi/2} 0 0</pose>
     <xacro:cylinder_inertia_sdf
         mass="${upper_mass}"

File: model/delta/parameters.xacro (robot description, xacro)
@@ -1,6 +1,6 @@
 <?xml version="1.0"?>
 <robot xmlns:xacro="http://www.ros.org/wiki/xacro" name="delta_parameters">
+<xacro:property name="base_depth" value="0.05"/>
 <xacro:property name="base_radius" value="0.3"/>
-<xacro:property name="base_depth" value="0.05"/>
 <xacro:property name="upper_length" value="0.3"/>
 <xacro:property name="upper_radius" value="0.01"/>
@@ -15,3 +15,9 @@
 <xacro:property name="end_effector_mass" value="0.05"/>
 <xacro:property name="break_indicator_radius" value="0.03"/>
+<xacro:property name="base_height"
+    value="${sqrt(lower_length**2 - (upper_length+base_radius-end_effector_radius)**2)}"
+/>
+<xacro:property name="lower_inclination"
+    value="${acos((upper_length+base_radius-end_effector_radius)/lower_length)}"
+/>
 </robot>

Commit message: Fixed gazebo model to world, works well.

File: model/delta/gazebo.sdf.xacro (robot description, xacro)
@@ -2,5 +2,20 @@
 <sdf version='1.4' xmlns:xacro="http://www.ros.org/wiki/xacro">
 <model name="delta">
-<static>false</static>
+<selfCollide>true</selfCollide>
+<joint name="world_fix" type="fixed">
+    <pose>0 0 0 0 0 0</pose>
+    <parent>world</parent>
+    <child>base</child>
+</joint>
+<physics>
+    <ode>
+        <island_threads>
+            3
+        </island_threads>
+        <solver>
+            <iters>50</iters>
+        </solver>
+    </ode>
+</physics>
 <xacro:include filename="parameters.xacro"/>
 <xacro:include filename="../macros/inertia.xacro"/>

File: model/delta/gazebo_joints/upper.sdf.xacro (robot description, xacro)
@@ -14,14 +14,4 @@
     </axis>
 </joint>
-<transmission name="theta_${number}_tran">
-    <type>transmission_interface/SimpleTransmission</type>
-    <joint name="theta_${number}">
-        <hardwareInterface>EffortJointInterface</hardwareInterface>
-    </joint>
-    <actuator name="theta_${number}">
-        <hardwareInterface>EffortJointInterface</hardwareInterface>
-        <mechanicalReduction>1</mechanicalReduction>
-    </actuator>
-</transmission>
 </xacro:macro>
 <xacro:joint_theta number="1" yaw="0"/>

File: model/delta/gazebo_links/base.sdf.xacro (robot description, xacro)
@@ -2,5 +2,5 @@
 <sdf xmlns:xacro="http://www.ros.org/wiki/xacro" name="base">
 <xacro:macro name="stand_part" params="number yaw">
-<visual name="stand_leg_${number}_visual">
+<visual name="stand_leg_${number}_visual_1">
     <pose>
         ${stand_radius*cos(yaw)}
@@ -10,10 +10,8 @@
     </pose>
     <geometry><box><size>
-                ${stand_leg_size}
-                ${stand_leg_size}
-                ${stand_height}
+        ${stand_leg_depth} ${stand_leg_width} ${stand_height}
     </size></box></geometry>
 </visual>
-<collision name="stand_leg_${number}_collision">
+<collision name="stand_leg_${number}_collision_1">
     <pose>
         ${stand_radius*cos(yaw)}
@@ -23,7 +21,5 @@
     </pose>
     <geometry><box><size>
-        ${stand_leg_size}
-        ${stand_leg_size}
-        ${-stand_height}
+        ${stand_leg_depth} ${stand_leg_depth} ${-stand_height}
     </size></box></geometry>
 </collision>
@@ -34,11 +30,55 @@
     </pose>
     <xacro:box_inertia_sdf
-        mass="${stand_mass}"
-        w="${stand_leg_size}"
-        h="${stand_leg_size}"
-        d="${stand_height}"
+        mass="${stand_vertical_mass}"
+        w="${stand_leg_depth}" h="${stand_leg_width}" d="${stand_height}"
     />
 </inertial>
-<visual name="stand_top_${number}_visual">
+<visual name="stand_leg_${number}_visual_2">
+    <pose>
+        ${stand_radius*cos(yaw)}
+        ${stand_radius*sin(yaw)}
+        ${-stand_height + stand_base_height/2}
+        0 0 ${yaw}
+    </pose>
+    <geometry>
+        <cylinder>
+            <length>${stand_base_height}</length>
+            <radius>${stand_base_radius}</radius>
+        </cylinder>
+    </geometry>
+</visual>
+<collision name="stand_leg_${number}_collision_2">
+    <pose>
+        ${stand_radius*cos(yaw)}
+        ${stand_radius*sin(yaw)}
+        ${-stand_height + stand_base_height/2}
+        0 0 ${yaw}
+    </pose>
+    <geometry>
+        <cylinder>
+            <length>${stand_base_height}</length>
+            <radius>${stand_base_radius}</radius>
+        </cylinder>
+    </geometry>
+    <surface>
+        <ode>
+            <mu>10</mu>
+            <mu2>10</mu2>
+            <slip>0</slip>
+            <slip2>0</slip2>
+        </ode>
+    </surface>
+</collision>
+<inertial>
+    <pose>
+        ${stand_radius*cos(yaw)} ${stand_radius*sin(yaw)} ${-stand_height+stand_base_height/2}
+        0 0 {yaw}
+    </pose>
+    <mass>${base_mass}</mass>
+    <xacro:cylinder_inertia_sdf
+        mass="${stand_base_mass}" radius="${stand_base_radius}" length="${stand_base_height}"
+    />
+</inertial>
+<visual name="stand_top_${number}_visual_3">
     <pose>
         ${0.5*(stand_radius+base_radius)*cos(yaw)}
@@ -49,9 +89,9 @@
     <geometry><box><size>
         ${stand_radius - base_radius}
-        ${stand_leg_size}
-        ${stand_leg_size}
+        ${stand_leg_width}
+        ${stand_leg_depth}
     </size></box></geometry>
 </visual>
-<collision name="stand_leg_base_${number}_collision">
+<collision name="stand_leg_base_${number}_collision_3">
     <pose>
         ${0.5*(stand_radius+base_radius)*cos(yaw)}
@@ -62,6 +102,6 @@
     <geometry><box><size>
         ${stand_radius - base_radius}
-        ${stand_leg_size}
-        ${stand_leg_size}
+        ${stand_leg_width}
+        ${stand_leg_depth}
     </size></box></geometry>
 </collision>
@@ -74,8 +114,8 @@
     </pose>
     <xacro:box_inertia_sdf
-        mass="${stand_mass}"
+        mass="${stand_horizontal_mass}"
         w="${stand_radius - base_radius}"
-        h="${stand_leg_size}"
-        d="${stand_leg_size}"
+        h="${stand_leg_width}"
+        d="${stand_leg_depth}"
     />
 </inertial>
@@ -99,4 +139,5 @@
     </geometry>
 </collision>
+<!--
 <inertial>
     <mass>${base_mass}</mass>
@@ -110,4 +151,5 @@
 <xacro:stand_part number="2" yaw="${pi}"/>
 <xacro:stand_part number="3" yaw="${-pi/3}"/>
+-->
 </link>
 </sdf>

File: model/delta/parameters.xacro (robot description, xacro)
@@ -1,23 +1,27 @@
 <?xml version="1.0"?>
 <robot xmlns:xacro="http://www.ros.org/wiki/xacro" name="delta_parameters">
-<xacro:property name="base_depth" value="0.05"/>
-<xacro:property name="base_radius" value="0.3"/>
+<xacro:property name="base_depth" value="0.02"/>
+<xacro:property name="base_radius" value="0.15"/>
 <xacro:property name="upper_length" value="0.3"/>
-<xacro:property name="upper_radius" value="0.01"/>
-<xacro:property name="lower_radius" value="0.01"/>
-<xacro:property name="lower_width" value="0.4"/>
+<xacro:property name="upper_radius" value="0.005"/>
+<xacro:property name="lower_radius" value="0.005"/>
+<xacro:property name="lower_width" value="0.1"/>
 <xacro:property name="lower_length" value="0.6"/>
-<xacro:property name="end_effector_radius" value="0.2"/>
-<xacro:property name="end_effector_depth" value="0.03"/>
-<xacro:property name="base_mass" value="0.1"/>
-<xacro:property name="upper_mass" value="0.04"/>
-<xacro:property name="lower_mass" value="0.06"/>
-<xacro:property name="end_effector_mass" value="0.05"/>
+<xacro:property name="end_effector_radius" value="0.1"/>
+<xacro:property name="end_effector_depth" value="0.01"/>
+<xacro:property name="base_mass" value="0.05"/>
+<xacro:property name="upper_mass" value="0.01"/>
+<xacro:property name="lower_mass" value="0.01"/>
+<xacro:property name="end_effector_mass" value="0.02"/>
 <xacro:property name="break_indicator_radius" value="0.03"/>
-<xacro:property name="stand_height" value="0.9"/>
-<xacro:property name="stand_radius" value="0.8"/>
-<xacro:property name="stand_leg_size" value="0.05"/>
-<xacro:property name="stand_mass" value="0.1"/>
+<xacro:property name="stand_height" value="1.1"/>
+<xacro:property name="stand_radius" value="1.2"/>
+<xacro:property name="stand_leg_width" value="0.1"/>
+<xacro:property name="stand_leg_depth" value="0.05"/>
+<xacro:property name="stand_horizontal_mass" value="0.01"/>
+<xacro:property name="stand_vertical_mass" value="0.01"/>
 <xacro:property name="stand_base_mass" value="1"/>
+<xacro:property name="stand_base_radius" value="0.12"/>
+<xacro:property name="stand_base_height" value="0.12"/>
 <xacro:property name="end_effector_height"
     value="${stand_height - sqrt(lower_length**2 - (upper_length+base_radius-end_effector_radius)**2)}"
