Commit message: Fixed urdf model and launch file

File: model/delta/ros_joints/upper.urdf.xacro (robot description, xacro)
@@ -1,4 +1,4 @@
 <?xml version="1.0"?>
-<robot xmlns:xacro="http://www.ros.org/wiki/xacro">
+<robot xmlns:xacro="http://www.ros.org/wiki/xacro" name="ros_links_upper">
 <!-- ===== THETA ===== -->
 <xacro:macro name="joint_theta" params="number yaw">
@@ -18,4 +18,5 @@
     <child link="upper_${number}"/>
 </joint>
+</xacro:macro>
 <xacro:joint_theta number="1" yaw="0"/>
 <xacro:joint_theta number="2" yaw="${pi*2/3}"/>
