Commit message: Added stand to gazebo model

File: model/delta/gazebo_links/base.sdf.xacro (robot description, xacro)
@@ -1,6 +1,86 @@
 <?xml version="1.0"?>
 <sdf xmlns:xacro="http://www.ros.org/wiki/xacro" name="base">
+<xacro:macro name="stand_part" params="number yaw">
+<visual name="stand_leg_${number}_visual">
+    <pose>
+        ${stand_radius*cos(yaw)}
+        ${stand_radius*sin(yaw)}
+        ${-stand_height/2}
+        0 0 ${yaw}
+    </pose>
+    <geometry><box><size>
+                ${stand_leg_size}
+                ${stand_leg_size}
+                ${stand_height}
+    </size></box></geometry>
+</visual>
+<collision name="stand_leg_${number}_collision">
+    <pose>
+        ${stand_radius*cos(yaw)}
+        ${stand_radius*sin(yaw)}
+        ${-stand_height/2}
+        0 0 ${yaw}
+    </pose>
+    <geometry><box><size>
+        ${stand_leg_size}
+        ${stand_leg_size}
+        ${-stand_height}
+    </size></box></geometry>
+</collision>
+<inertial>
+    <pose>
+        ${stand_radius*cos(yaw)} ${stand_radius*sin(yaw)} ${-stand_height/2}
+        0 0 {yaw}
+    </pose>
+    <xacro:box_inertia_sdf
+        mass="${stand_mass}"
+        w="${stand_leg_size}"
+        h="${stand_leg_size}"
+        d="${stand_height}"
+    />
+</inertial>
+<visual name="stand_top_${number}_visual">
+    <pose>
+        ${0.5*(stand_radius+base_radius)*cos(yaw)}
+        ${0.5*(stand_radius+base_radius)*sin(yaw)}
+        0
+        0 0 ${yaw}
+    </pose>
+    <geometry><box><size>
+        ${stand_radius - base_radius}
+        ${stand_leg_size}
+        ${stand_leg_size}
+    </size></box></geometry>
+</visual>
+<collision name="stand_leg_base_${number}_collision">
+    <pose>
+        ${0.5*(stand_radius+base_radius)*cos(yaw)}
+        ${0.5*(stand_radius+base_radius)*sin(yaw)}
+        0
+        0 0 ${yaw}
+    </pose>
+    <geometry><box><size>
+        ${stand_radius - base_radius}
+        ${stand_leg_size}
+        ${stand_leg_size}
+    </size></box></geometry>
+</collision>
+<inertial>
+    <pose>
+        ${0.5*(stand_radius+base_radius)*cos(yaw)}
+        ${0.5*(stand_radius+base_radius)*sin(yaw)}
+        0
+        0 0 ${yaw}
+    </pose>
+    <xacro:box_inertia_sdf
+        mass="${stand_mass}"
+        w="${stand_radius - base_radius}"
+        h="${stand_leg_size}"
+        d="${stand_leg_size}"
+    />
+</inertial>
+</xacro:macro>
 <link name="base">
-<pose> 0 0 ${base_height} 0 0 0</pose>
+<pose> 0 0 ${stand_height} 0 0 0</pose>
 <visual name="base_visual">
     <geometry>
@@ -27,4 +107,7 @@
     />
 </inertial>
+<xacro:stand_part number="1" yaw="${pi/3}"/>
+<xacro:stand_part number="2" yaw="${pi}"/>
+<xacro:stand_part number="3" yaw="${-pi/3}"/>
 </link>
 </sdf>

File: model/delta/gazebo_links/end_effector.sdf.xacro (robot description, xacro)
@@ -32,5 +32,5 @@
 </xacro:macro>
 <link name="end_effector">
-<pose> 0 0 0 0 0 0</pose>
+<pose> 0 0 ${end_effector_height} 0 0 0</pose>
 <visual name="end_effector_visual">
     <pose>0 0 0 0 0 0</pose>

File: model/delta/gazebo_links/lower.sdf.xacro (robot description, xacro)
@@ -7,5 +7,5 @@
     ${(base_radius + upper_length)*cos(yaw) - (lower_width/2)*sin(yaw)}
     ${(base_radius + upper_length)*sin(yaw) + (lower_width/2)*cos(yaw)}
-    ${base_height}
+    ${stand_height}
     0 ${pi - lower_inclination} ${yaw}
 </pose>
@@ -48,5 +48,5 @@
     ${(base_radius + upper_length)*cos(yaw) + (lower_width/2)*sin(yaw)}
     ${(base_radius + upper_length)*sin(yaw) - (lower_width/2)*cos(yaw)}
-    ${base_height}
+    ${stand_height}
     0 ${pi - lower_inclination} ${yaw}
 </pose>

File: model/delta/gazebo_links/upper.sdf.xacro (robot description, xacro)
@@ -4,5 +4,5 @@
 <link name="upper_${number}">
 <pose>
-    ${base_radius*cos(yaw)} ${base_radius*sin(yaw)} ${base_height}
+    ${base_radius*cos(yaw)} ${base_radius*sin(yaw)} ${stand_height}
     0 0 ${yaw}
 </pose>

File: model/delta/parameters.xacro (robot description, xacro)
@@ -15,6 +15,11 @@
 <xacro:property name="end_effector_mass" value="0.05"/>
 <xacro:property name="break_indicator_radius" value="0.03"/>
-<xacro:property name="base_height"
-    value="${sqrt(lower_length**2 - (upper_length+base_radius-end_effector_radius)**2)}"
+<xacro:property name="stand_height" value="0.9"/>
+<xacro:property name="stand_radius" value="0.8"/>
+<xacro:property name="stand_leg_size" value="0.05"/>
+<xacro:property name="stand_mass" value="0.1"/>
+<xacro:property name="stand_base_mass" value="1"/>
+<xacro:property name="end_effector_height"
+    value="${stand_height - sqrt(lower_length**2 - (upper_length+base_radius-end_effector_radius)**2)}"
 />
 <xacro:property name="lower_inclination"

File: model/macros/inertia.xacro (robot description, xacro)
@@ -17,3 +17,11 @@
 </inertia>
 </xacro:macro>
+<xacro:macro name="box_inertia_sdf" params="mass w h d">
+<inertia>
+    <ixx>${mass*(h**2 + d**2)/12}</ixx>
+    <iyy>${mass*(w**2 + d**2)/12}</iyy>
+    <izz>${mass*(w**2 + h**2)/12}</izz>
+    <ixy>0</ixy> <ixz>0</ixz> <iyz>0</iyz>
+</inertia>
+</xacro:macro>
 </robot>
